File: draft5_4lyr.sch (EAGLE design)
At the start: 179 parts, among them Q1 Si2333, Q2 2N7002, Q3 2N7002, Q4 2N7002, Q5 2N7002, Q6 2N7002, Q7 2N7002, SW1 TOUCH_PAD-CIRCLE-15MM, SW10 TOUCH_PAD-CIRCLE-15MM, SW4 TOUCH_PAD-CIRCLE-15MM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

Commit message: Added JTAG header
Parts:
- removed R6: 100K, rcl:R-US_R0603
- added JTAG: HEADER-10P-SMD-MALE2, 00-EvaLibrary:HEADER-10P-SMD-MALE2
- added R11, R14, R45, R46: 100K, rcl:R-US_R0603
Connections:
- new net TCK: JTAG.4, R14.1, U7B.PB28
- new net TDI: JTAG.8, R45.1, U7B.PB29
- new net TDO: JTAG.6, U7B.PB30
- new net TMS: JTAG.2, R11.1, U7B.PB31
- net !RESET: now also JTAG.10, R46.1
- net !SD_CARD: now also U7C.PC8; no longer R6.2, U7C.PC9
- net AVR_PWR: now also JTAG.1, R11.2, R14.2, R45.2, R46.2; no longer R6.1
- net CS_SD: now also U7C.PC9; no longer U7C.PC8
- net GND: now also JTAG.3, JTAG.5, JTAG.9
Other:
- note added: "Ensure pull-up on !SD_CARD"

Commit message: Added USB enumeration sense
Connections:
- removed net N$24: R7.1, U1.AD2/GIO9
- new net USB_SENSE: R7.1, U1.AD2/GIO9, U7D.PD6
Changed lines of the file:
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@@
 </segment>
 </net>
-<net name="N$24" class="0">
+<net name="USB_SENSE" class="0">
 <segment>
 <wire x1="-167.64" y1="-29.21" x2="-165.1" y2="-29.21" width="0.1524" layer="91"/>
 <pinref part="R7" gate="G$1" pin="1"/>
 <pinref part="U1" gate="G$1" pin="AD2/GIO9"/>
+<wire x1="-165.1" y1="-29.21" x2="-165.1" y2="-35.56" width="0.1524" layer="91"/>
+<junction x="-165.1" y="-29.21"/>
+<label x="-165.1" y="-35.56" size="1.778" layer="95" rot="R270" xref="yes"/>
+</segment>
+<segment>
+<pinref part="U7" gate="D" pin="PD6"/>
+<wire x1="600.71" y1="-273.05" x2="595.63" y2="-273.05" width="0.1524" layer="91"/>
+<label x="595.63" y="-273.05" size="1.778" layer="95" rot="R180" xref="yes"/>
 </segment>
 </net>
