File: prototype_board.sch (EAGLE design)
At the start: 183 parts, among them Q1 Si2333, Q2 2N7002, Q3 2N7002, Q4 2N7002, Q5 2N7002, Q6 2N7002, Q7 2N7002, SW1 TOUCH_PAD-CIRCLE-15MM, SW10 TOUCH_PAD-CIRCLE-15MM, SW4 TOUCH_PAD-CIRCLE-15MM, SW5 TOUCH_PAD-CIRCLE-15MM, SW6 TOUCH_PAD-CIRCLE-15MM, SW7 TOUCH_PAD-CIRCLE-15MM, SW8 TOUCH_PAD-CIRCLE-15MM, SW9 TOUCH_PAD-CIRCLE-15MM, U1 CC8531, U2 CC2591, U3 TLV320AIC3204, U6 LTC4088-2, U7 ATSAM3X8E_ALT-LQFP-144, U8 AT42QT1110-TQFP, U9 LM4881, X1 48MHz, X3 12MHz

Commit message: Fixed stuff, created prototype board
Parts:
- removed C57: 2.2u, rcl:C-EUC0603
- removed L19: BEAD, SparkFun-Passives:INDUCTOR0603
- removed MICROSD: MICROSD104031-0811, 00-EvaLibrary:MICROSD104031-0811
- removed R28, R29, R30: 0, 00-EvaLibrary:R-US_R0603
- removed TO_AUX1, TO_AUX2: HEADER-10P-SMD-2MM-FEMALE, 00-EvaLibrary:HEADER-10P-SMD-2MM-FEMALE
- removed TO_MAIN1, TO_MAIN2: HEADER-10P-SMD-2MM-MALE, 00-EvaLibrary:HEADER-10P-SMD-2MM-MALE
- added !CHANGE, !PAIR, !SD_CARD, AMP_VDD, AUDIO, AUX_VDD, AVDD, AVDD_CODEC, AVR_VDD, BCLK, BCLK2, BLUE_BOT, BLUE_TOP, CS_CC8531, CS_CODEC, CS_SD, CS_TOUCH, DIN, DIN2, DOUT, DOUT2, DVDD_CODEC, GREEN_BOT, GREEN_TOP, IOVDD, LINEIN_SENSE, LINE_L, LINE_R, MCLK, MISO, MISO2, MISO3, MISO4, MOSI, MOSI2, MOSI3, MOSI4, PHONE_L, PHONE_R, PHONE_SENSE, RED_BOT, RED_TOP, RESET_CC8531, RESET_CODEC, SCLK, SCLK2, SCLK3, SCLK4, USB_SENSE, VDD_SD, WCLK, WCLK2: SOLDERJUMPERNO, SparkFun-Passives (1):SOLDERJUMPERNO
- added AVR1, AVR2: (no value), SparkFun-LED:LED1206
- added MICROSD1: MICROSD104031-0811, 00-EvaLibrary:MICROSD104031-0811
- added R6: 100, rcl:R-US_R0603
- EXT: value 0 -> SOLDERJUMPERNO; device rcl:R-US_R0603 -> SparkFun-Passives (1):SOLDERJUMPERNO
- R27: value 0 -> 100; device 00-EvaLibrary:R-US_R0603 -> rcl:R-US_R0603
Connections:
- removed net AVR_PWR: C35.1, C46.1, C47.1, C69.1, ERASE.3, JTAG.1, L16.1, MICROSD.VDD, R11.2, R14.2, R43.1, R44.2, R45.2, R46.2, U7P.VDDANA, U7P.VDDBU, U7P.VDDIN, U7P.VDDIO_1, U7P.VDDIO_2, U7P.VDDIO_3, U7P.VDDIO_4, U7P.VDDUTMI, U7X.ADVREF
- removed net M_BLCK: U7A.PA14
- new net !AVR_LED2: AVR1.C, U7B.PB27
- new net !AVR_LED3: AVR2.C, U7A.PA19
- new net AVR_VDD: C35.1, C46.1, C47.1, C69.1, ERASE.3, JTAG.1, L16.1, R11.2, R14.2, R27.2, R43.1, R44.2, R45.2, R46.2, R6.2, U7P.VDDANA, U7P.VDDBU, U7P.VDDIN, U7P.VDDIO_1, U7P.VDDIO_2, U7P.VDDIO_3, U7P.VDDIO_4, U7P.VDDUTMI, U7X.ADVREF, VDD_SD.2
- new net C_AUDIO: AUDIO.1, C36.1, R12.1, U9.OUTA
- new net C_CS_CODEC: CS_CODEC.1, U3.SCL/SSZ
- new net C_LINEIN_SENSE: LINEIN_SENSE.1, LINE_IN.L_SW, R22.1
- new net C_MISO: MISO2.1, U3.MISO/MFP4
- new net C_MOSI: MOSI2.1, U3.SDA/MOSI
- new net C_PHONE_SENSE: PHONE_OUT.L_SW, PHONE_SENSE.1, R24.1
- new net C_RESET_CODEC: RESET_CODEC.1, U3.!RESET
- new net C_SCLK: SCLK2.1, U3.SCLK/MFP3
- new net M_BCLK: BCLK2.2, U7A.PA14
- new net N$20: AVDD.1, L2.2
- new net N$24: IOVDD.1, L1.2
- new net N$39: AVDD_CODEC.1, L14.2
- new net N$46: DVDD_CODEC.1, L15.2
- new net N$47: AUX_VDD.1, L18.2
- new net N$52: AMP_VDD.1, L3.2
- new net N$57: CS_SD.2, MICROSD1.!CS
- new net N$88: MICROSD1.MISO, MISO4.2
- new net N$89: !SD_CARD.2, MICROSD1.SWA
- new net N$91: MICROSD1.VDD, VDD_SD.1
- new net N$92: AVR_VDD.1, L16.2
- new net N$93: AVR1.A, R6.1
- new net N$94: AVR2.A, R27.1
- new net X_!PAIR: !PAIR.1, U1.GIO1
- new net X_BCLK: BCLK.1, L6.1
- new net X_CS_CC8531: CC_DEBUG.5, CS_CC8531.1, U1.CSN
- new net X_DIN: DIN.1, L13.1
- new net X_DOUT: DOUT.1, L11.1
- new net X_MCLK: L5.1, MCLK.1
- new net X_MISO: CC_DEBUG.10, MISO.1, U1.MISO
- new net X_MOSI: CC_DEBUG.8, MOSI.1, U1.MOSI
- new net X_RESET_CC8531: CC_DEBUG.7, L4.2, RESET_CC8531.1
- new net X_SCLK: CC_DEBUG.6, SCLK.1, U1.SCLK
- new net X_USB_SENSE: R7.1, U1.AD2/GIO9, USB_SENSE.1
- new net X_WCLK: L9.1, WCLK.1
- net !CHANGE: now also !CHANGE.2; no longer TO_AUX1.9
- net !PAIR: now also !PAIR.2; no longer U1.GIO1
- net !SD_CARD: now also !SD_CARD.1; no longer MICROSD.SWA
- net 3.3V: now also AMP_VDD.2, AUX_VDD.2, AVDD.2, AVDD_CODEC.2, AVR_VDD.2, DVDD_CODEC.2, EXT.1, IOVDD.2; no longer EXT.2, L1.2, L14.2, L15.2, L16.2, L18.2, L19.2, L2.2, L3.2
- net AUDIO: now also AUDIO.2; no longer C36.1, R12.1, U9.OUTA
- net AUX_!CHANGE: now also !CHANGE.1; no longer TO_MAIN1.10
- net AUX_BLUE_BOT: now also BLUE_BOT.1; no longer TO_MAIN2.7
- net AUX_BLUE_TOP: now also BLUE_TOP.1; no longer TO_MAIN2.4
- net AUX_CS: now also CS_TOUCH.1; no longer TO_MAIN1.8
- net AUX_GREEN_BOT: now also GREEN_BOT.1; no longer TO_MAIN2.5
- net AUX_GREEN_TOP: now also GREEN_TOP.1; no longer TO_MAIN2.6
- net AUX_MISO: now also MISO3.1; no longer TO_MAIN1.4
- net AUX_MOSI: now also MOSI3.1; no longer TO_MAIN1.6
- net AUX_RED_BOT: now also RED_BOT.1; no longer TO_MAIN2.3
- net AUX_RED_TOP: now also RED_TOP.1; no longer TO_MAIN2.8
- net AUX_SCLK: now also SCLK3.1; no longer TO_MAIN1.2
- net AUX_VDD: now also C65.1, L18.1; no longer TO_MAIN1.1, TO_MAIN1.3, TO_MAIN1.5, TO_MAIN2.1, TO_MAIN2.2
- net AUX_VSS: no longer TO_MAIN1.7, TO_MAIN1.9, TO_MAIN2.10, TO_MAIN2.9
- net BCLK: now also BCLK.2, BCLK2.1; no longer L6.1
- net BLUE_BOT: now also BLUE_BOT.2; no longer TO_AUX2.8
- net BLUE_TOP: now also BLUE_TOP.2; no longer TO_AUX2.3
- net CS_CC8531: now also CS_CC8531.2; no longer CC_DEBUG.5, U1.CSN
- net CS_CODEC: now also CS_CODEC.2; no longer U3.SCL/SSZ
- net CS_SD: now also CS_SD.1; no longer MICROSD.!CS
- net CS_TOUCH: now also CS_TOUCH.2; no longer TO_AUX1.7
- net DIN: now also DIN.2, DOUT2.1; no longer L13.1
- net DOUT: now also DIN2.1, DOUT.2; no longer L11.1
- net GND: now also MICROSD1.GND, MICROSD1.SWB; no longer C57.2, MICROSD.GND, MICROSD.SWB, TO_AUX1.10, TO_AUX1.6, TO_AUX1.8, TO_AUX2.10, TO_AUX2.9
- net GREEN_BOT: now also GREEN_BOT.2; no longer TO_AUX2.6
- net GREEN_TOP: now also GREEN_TOP.2; no longer TO_AUX2.5
- net LINEIN_SENSE: now also LINEIN_SENSE.2; no longer LINE_IN.L_SW, R22.1
- net LINE_L: now also LINE_L.1; no longer R27.1
- net LINE_R: now also LINE_R.1; no longer R29.1
- net MCLK: now also MCLK.2; no longer L5.1
- net MISO: now also MISO.2, MISO2.2, MISO3.2, MISO4.1; no longer CC_DEBUG.10, MICROSD.MISO, TO_AUX1.3, U1.MISO, U3.MISO/MFP4
- net MOSI: now also MOSI.2, MOSI2.2, MOSI3.2, MOSI4.1; no longer CC_DEBUG.8, MICROSD.MOSI, TO_AUX1.5, U1.MOSI, U3.SDA/MOSI
- net M_DIN/S_DOUT: now also DIN2.2
- net M_DOUT/S_DIN: now also DOUT2.2
- net M_WCLK: now also WCLK2.2
- net N$43: now also LINE_L.2, PHONE_L.2; no longer R27.2, R28.2
- net N$45: now also LINE_R.2, PHONE_R.2; no longer R29.2, R30.2
- net N$50: now also EXT.2; no longer EXT.1
- net N$67: now also MICROSD1.SCLK, SCLK4.2; no longer C57.1, L19.1, TO_AUX2.1, TO_AUX2.2
- net N$84: now also MICROSD1.MOSI, MOSI4.2; no longer C65.1, L18.1, TO_AUX1.2, TO_AUX1.4
- net PHONE_L: now also PHONE_L.1; no longer R28.1
- net PHONE_R: now also PHONE_R.1; no longer R30.1
- net PHONE_SENSE: now also PHONE_SENSE.2; no longer PHONE_OUT.L_SW, R24.1
- net RED_BOT: now also RED_BOT.2; no longer TO_AUX2.4
- net RED_TOP: now also RED_TOP.2; no longer TO_AUX2.7
- net RESET_CC8531: now also RESET_CC8531.2; no longer CC_DEBUG.7, L4.2
- net RESET_CODEC: now also RESET_CODEC.2; no longer U3.!RESET
- net SCLK: now also SCLK.2, SCLK2.2, SCLK3.2, SCLK4.1; no longer CC_DEBUG.6, MICROSD.SCLK, TO_AUX1.1, U1.SCLK, U3.SCLK/MFP3
- net USB_SENSE: now also USB_SENSE.2; no longer R7.1, U1.AD2/GIO9
- net WCLK: now also WCLK.2, WCLK2.1; no longer L9.1
Other:
- moved on the sheet: C65, L18, R27
