File: prototype_board.brd (EAGLE design)
At the start: 200 x 200 mm, 229 parts, among them Q1 Si2333, Q2 2N7002, Q3 2N7002, Q4 2N7002, Q5 2N7002, Q6 2N7002, Q7 2N7002, SW1 TOUCH_PAD-CIRCLE-15MM, SW10 TOUCH_PAD-CIRCLE-15MM, SW4 TOUCH_PAD-CIRCLE-15MM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

Commit message: New revision, changed proto board
Parts:
- added C57, C70: 0.47u, rcl:C0603
- moved AMP_VDD 164.6 mm to (180.3, -21.7)
- moved AVDD 164.6 mm to (176.8, -28.2)
- moved C1 164.6 mm to (155.5, -37.0)
- moved C10 164.6 mm to (172.0, -42.5)
- moved C11 164.6 mm to (166.0, -48.0)
- moved C12 164.6 mm to (173.0, -50.0)
- moved C15 164.6 mm to (202.5, -17.5)
- moved C16 164.6 mm to (214.5, -22.5)
- moved C17 164.6 mm to (210.5, -25.5)
- moved C18 164.6 mm to (208.0, -31.0)
- moved C19 164.6 mm to (205.0, -27.5)
- moved C2 164.6 mm to (149.5, -33.0)
- moved C20 164.6 mm to (216.5, -31.0)
- moved C21 164.6 mm to (216.0, -27.0)
- moved C22 164.6 mm to (219.0, -33.5)
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Connections:
- new net N$95: C57.2, R13.2
- new net N$96: C70.2, R16.2
- net N$43: now also C57.1; no longer R13.2
- net N$45: now also C70.1; no longer R16.2
Routing:
- net RED_TOP: track 0.00 -> 102.0 mm
- net GREEN_TOP: track 0.00 -> 100.3 mm
- net N$61: track 0.00 -> 99.8 mm
- net RED_BOT: track 0.00 -> 98.6 mm, vias 0 -> 2
- net BLUE_TOP: track 0.00 -> 97.7 mm
- net GREEN_BOT: track 0.00 -> 96.1 mm, vias 0 -> 2
- net BLUE_BOT: track 0.00 -> 92.8 mm
- net N$44: track 0.00 -> 90.2 mm
- net N$63: track 0.00 -> 86.0 mm
- net N$70: track 0.00 -> 84.0 mm
- net BCLK: track 0.00 -> 61.7 mm, vias 0 -> 2
- net SCLK: track 44.3 -> 105.2 mm, vias 2 -> 4
- net PHONE_SENSE: track 0.00 -> 60.9 mm, vias 0 -> 2
- net WCLK: track 0.00 -> 58.0 mm, vias 0 -> 2
- net MISO: track 37.7 -> 94.8 mm, vias 2 -> 5
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Other:
- board size 200 x 200 mm -> 200 x 114 mm
