File: prototype_rev2.sch (EAGLE design)
At the start: 231 parts, among them Q1 Si2333, Q2 2N7002, Q3 2N7002, Q4 2N7002, Q5 2N7002, Q6 2N7002, Q7 2N7002, SW1 TOUCH_PAD-CIRCLE-15MM, SW10 TOUCH_PAD-CIRCLE-15MM, SW4 TOUCH_PAD-CIRCLE-15MM, SW5 TOUCH_PAD-CIRCLE-15MM, SW6 TOUCH_PAD-CIRCLE-15MM, SW7 TOUCH_PAD-CIRCLE-15MM, SW8 TOUCH_PAD-CIRCLE-15MM, SW9 TOUCH_PAD-CIRCLE-15MM, U1 CC8531, U2 CC2591, U3 TLV320AIC3204, U6 LTC4088-2, U7 ATSAM3X8E_ALT-LQFP-144, U8 AT42QT1110-TQFP, U9 LM4881, X1 48MHz, X3 12MHz

Commit message: New revision, changed proto board
Parts:
- removed AMP_VDD, AVDD, AVDD_CODEC, BCLK2, CS_CC8531, CS_CODEC, CS_SD, CS_TOUCH, DIN2, DOUT2, DVDD_CODEC, IOVDD, MCLK, MISO, MISO2, MISO3, MISO4, MOSI, MOSI2, MOSI3, MOSI4, RESET_CC8531, RESET_CODEC, SCLK, SCLK2, SCLK3, SCLK4, VDD_SD, WCLK2: SOLDERJUMPERNO, SparkFun-Passives (1):SOLDERJUMPERNO
- removed R17: 0, rcl:R-US_R0603
- removed R27: 100, rcl:R-US_R0603
- added AMP_AVDD, AUX_CS, AUX_MISO, AUX_MOSI, AUX_SCLK, CC8531_AVDD, CC8531_BCLK, CC8531_CS, CC8531_DIN, CC8531_DOUT, CC8531_IOVDD, CC8531_MCLK, CC8531_MISO, CC8531_MOSI, CC8531_RESET, CC8531_SCLK, CC8531_WCLK, CODEC_AVDD, CODEC_CS, CODEC_DVDD, CODEC_MISO, CODEC_MOSI, CODEC_RESET, CODEC_SCLK, SD_CS, SD_MISO, SD_MOSI, SD_SCLK, SD_VDD: 2P-HEADER-JUMPER, SparkFun-Connectors:2P-HEADER-JUMPER
- added R47: 100, rcl:R-US_R0603
- !CHANGE, !PAIR, !SD_CARD, AUDIO, AUX_VDD, AVR_VDD, BCLK, BLUE_BOT, BLUE_TOP, DIN, DOUT, EXT, GREEN_BOT, GREEN_TOP, LINEIN_SENSE, LINE_L, LINE_R, PHONE_L, PHONE_R, PHONE_SENSE, RED_BOT, RED_TOP, USB_SENSE, WCLK: value SOLDERJUMPERNO -> 2P-HEADER-JUMPER; device SparkFun-Passives (1):SOLDERJUMPERNO -> SparkFun-Connectors:2P-HEADER-JUMPER
- renumbered C57 to C71
Connections:
- removed net N$20 (its old number): AVDD.1, L2.2
- removed net N$24 (its old number): IOVDD.1, L1.2
- new net N$95: CODEC_AVDD.P$1, L14.2
- new net N$96: CODEC_DVDD.P$1, L15.2
- net !CHANGE: now also !CHANGE.P$2; no longer !CHANGE.2
- net !PAIR: now also !PAIR.P$2; no longer !PAIR.2
- net !SD_CARD: now also !SD_CARD.P$1; no longer !SD_CARD.1
- net 3.3V: now also AMP_AVDD.P$2, AUX_VDD.P$2, AVR_VDD.P$2, CC8531_AVDD.P$2, CC8531_IOVDD.P$2, CODEC_AVDD.P$2, CODEC_DVDD.P$2, EXT.P$1; no longer AMP_VDD.2, AUX_VDD.2, AVDD.2, AVDD_CODEC.2, AVR_VDD.2, DVDD_CODEC.2, EXT.1, IOVDD.2
- net AGND: no longer R17.2
- net AUDIO: now also AUDIO.P$2; no longer AUDIO.2
- net AUX_!CHANGE: now also !CHANGE.P$1; no longer !CHANGE.1
- net AUX_BLUE_BOT: now also BLUE_BOT.P$1; no longer BLUE_BOT.1
- net AUX_BLUE_TOP: now also BLUE_TOP.P$1; no longer BLUE_TOP.1
- net AUX_CS: now also AUX_CS.P$1; no longer CS_TOUCH.1
- net AUX_GREEN_BOT: now also GREEN_BOT.P$1; no longer GREEN_BOT.1
- net AUX_GREEN_TOP: now also GREEN_TOP.P$1; no longer GREEN_TOP.1
- net AUX_MISO: now also AUX_MISO.P$1; no longer MISO3.1
- net AUX_MOSI: now also AUX_MOSI.P$1; no longer MOSI3.1
- net AUX_RED_BOT: now also RED_BOT.P$1; no longer RED_BOT.1
- net AUX_RED_TOP: now also RED_TOP.P$1; no longer RED_TOP.1
- net AUX_SCLK: now also AUX_SCLK.P$1; no longer SCLK3.1
- net AVR_VDD: now also R47.2, SD_VDD.P$2; no longer R27.2, VDD_SD.2
- net BCLK: now also BCLK.P$1, CC8531_BCLK.P$2; no longer BCLK.2, BCLK2.1
- net BLUE_BOT: now also BLUE_BOT.P$2; no longer BLUE_BOT.2
- net BLUE_TOP: now also BLUE_TOP.P$2; no longer BLUE_TOP.2
- net CS_CC8531: now also CC8531_CS.P$2; no longer CS_CC8531.2
- net CS_CODEC: now also CODEC_CS.P$2; no longer CS_CODEC.2
- net CS_SD: now also SD_CS.P$1; no longer CS_SD.1
- net CS_TOUCH: now also AUX_CS.P$2; no longer CS_TOUCH.2
- net C_AUDIO: now also AUDIO.P$1; no longer AUDIO.1
- net C_CS_CODEC: now also CODEC_CS.P$1; no longer CS_CODEC.1
- net C_LINEIN_SENSE: now also LINEIN_SENSE.P$1; no longer LINEIN_SENSE.1
- net C_MISO: now also CODEC_MISO.P$1; no longer MISO2.1
- net C_MOSI: now also CODEC_MOSI.P$1; no longer MOSI2.1
- net C_PHONE_SENSE: now also PHONE_SENSE.P$1; no longer PHONE_SENSE.1
- net C_RESET_CODEC: now also CODEC_RESET.P$1; no longer RESET_CODEC.1
- net C_SCLK: now also CODEC_SCLK.P$1; no longer SCLK2.1
- net DIN: now also CC8531_DIN.P$2, DIN.P$1; no longer DIN.2, DOUT2.1
- net DOUT: now also CC8531_DOUT.P$2, DOUT.P$1; no longer DIN2.1, DOUT.2
- net GND: no longer R17.1
- net GREEN_BOT: now also GREEN_BOT.P$2; no longer GREEN_BOT.2
- net GREEN_TOP: now also GREEN_TOP.P$2; no longer GREEN_TOP.2
- net LINEIN_SENSE: now also LINEIN_SENSE.P$2; no longer LINEIN_SENSE.2
- net LINE_L: now also LINE_L.P$1; no longer LINE_L.1
- net LINE_R: now also LINE_R.P$1; no longer LINE_R.1
- net MCLK: now also CC8531_MCLK.P$2; no longer MCLK.2
- net MISO: now also AUX_MISO.P$2, CC8531_MISO.P$2, CODEC_MISO.P$2, SD_MISO.P$1; no longer MISO.2, MISO2.2, MISO3.2, MISO4.1
- net MOSI: now also AUX_MOSI.P$2, CC8531_MOSI.P$2, CODEC_MOSI.P$2, SD_MOSI.P$1; no longer MOSI.2, MOSI2.2, MOSI3.2, MOSI4.1
- net M_BCLK: now also BCLK.P$2; no longer BCLK2.2
- net M_DIN/S_DOUT: now also DOUT.P$2; no longer DIN2.2
- net M_DOUT/S_DIN: now also DIN.P$2; no longer DOUT2.2
- net M_WCLK: now also WCLK.P$2; no longer WCLK2.2
- net N$39: now also MICROSD1.!CS, SD_CS.P$2; no longer AVDD_CODEC.1, L14.2
- net N$43: now also LINE_L.P$2, PHONE_L.P$2; no longer LINE_L.2, PHONE_L.2
- net N$45: now also LINE_R.P$2, PHONE_R.P$2; no longer LINE_R.2, PHONE_R.2
- net N$46: now also MICROSD1.SCLK, SD_SCLK.P$2; no longer DVDD_CODEC.1, L15.2
- net N$47: now also MICROSD1.MOSI, SD_MOSI.P$2; no longer AUX_VDD.1, L18.2
- net N$50: now also EXT.P$2; no longer EXT.2
- net N$52: now also MICROSD1.MISO, SD_MISO.P$2; no longer AMP_VDD.1, L3.2
- net N$57: now also !SD_CARD.P$2, MICROSD1.SWA; no longer CS_SD.2, MICROSD1.!CS
- net N$67: now also MICROSD1.VDD, SD_VDD.P$1; no longer MICROSD1.SCLK, SCLK4.2
- net N$84: now also AVR_VDD.P$1, L16.2; no longer MICROSD1.MOSI, MOSI4.2
- net N$88: now also AUX_VDD.P$1, L18.2; no longer MICROSD1.MISO, MISO4.2
- net N$89: now also AMP_AVDD.P$1, L3.2; no longer !SD_CARD.2, MICROSD1.SWA
- net N$91: now also CC8531_AVDD.P$1, L2.2; no longer MICROSD1.VDD, VDD_SD.1
- net N$92: now also CC8531_IOVDD.P$1, L1.2; no longer AVR_VDD.1, L16.2
- net N$94: now also R47.1; no longer R27.1
- net PHONE_L: now also PHONE_L.P$1; no longer PHONE_L.1
- net PHONE_R: now also PHONE_R.P$1; no longer PHONE_R.1
- net PHONE_SENSE: now also PHONE_SENSE.P$2; no longer PHONE_SENSE.2
- net RED_BOT: now also RED_BOT.P$2; no longer RED_BOT.2
- net RED_TOP: now also RED_TOP.P$2; no longer RED_TOP.2
- net RESET_CC8531: now also CC8531_RESET.P$2; no longer RESET_CC8531.2
- net RESET_CODEC: now also CODEC_RESET.P$2; no longer RESET_CODEC.2
- net SCLK: now also AUX_SCLK.P$2, CC8531_SCLK.P$2, CODEC_SCLK.P$2, SD_SCLK.P$1; no longer SCLK.2, SCLK2.2, SCLK3.2, SCLK4.1
- net USB_SENSE: now also USB_SENSE.P$2; no longer USB_SENSE.2
- net WCLK: now also CC8531_WCLK.P$2, WCLK.P$1; no longer WCLK.2, WCLK2.1
- net X_!PAIR: now also !PAIR.P$1; no longer !PAIR.1
- net X_BCLK: now also CC8531_BCLK.P$1; no longer BCLK.1
- net X_CS_CC8531: now also CC8531_CS.P$1; no longer CS_CC8531.1
- net X_DIN: now also CC8531_DIN.P$1; no longer DIN.1
- net X_DOUT: now also CC8531_DOUT.P$1; no longer DOUT.1
- net X_MCLK: now also CC8531_MCLK.P$1; no longer MCLK.1
- net X_MISO: now also CC8531_MISO.P$1; no longer MISO.1
- net X_MOSI: now also CC8531_MOSI.P$1; no longer MOSI.1
- net X_RESET_CC8531: now also CC8531_RESET.P$1; no longer RESET_CC8531.1
- net X_SCLK: now also CC8531_SCLK.P$1; no longer SCLK.1
- net X_USB_SENSE: now also USB_SENSE.P$1; no longer USB_SENSE.1
- net X_WCLK: now also CC8531_WCLK.P$1; no longer WCLK.1
Other:
- moved on the sheet: AVR1, AVR2, C65, C70, L18, MICROSD1, R16, R6
