File: prototype_rev2.brd (EAGLE design)
At the start: 242 parts, among them Q1 Si2333, Q2 2N7002, Q3 2N7002, Q4 2N7002, Q5 2N7002, Q6 2N7002, Q7 2N7002, SW1 TOUCH_PAD-CIRCLE-15MM, SW10 TOUCH_PAD-CIRCLE-15MM, SW4 TOUCH_PAD-CIRCLE-15MM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

Commit message: Board layout work
Parts:
- removed U$11, U$13, U$6, U$7: (no value), 00-EvaLibrary:STANDOFF_3/16
- moved PHONE_R 574.5 mm to (133.8, 23.8), turned to 270 degrees
- moved LINE_R 566.5 mm to (130.8, 23.8), turned to 270 degrees
- moved PHONE_L 553.3 mm to (113.5, 23.5), turned to 270 degrees
- moved LINE_L 545.2 mm to (110.5, 23.5), turned to 270 degrees
- moved SD_VDD 514.5 mm to (65.5, 65.2), turned to 270 degrees
- moved !SD_CARD 493.5 mm to (50.2, 55.0), turned to 90 degrees
- moved SD_MISO 489.5 mm to (62.2, 55.2), turned to 90 degrees
- moved SD_MOSI 480.7 mm to (56.2, 55.2), turned to 90 degrees
- moved SD_SCLK 474.3 mm to (59.2, 55.2), turned to 90 degrees
- moved AMP_AVDD 471.6 mm to (154.5, -38.5)
- moved AUX_VDD 471.6 mm to (154.5, -31.0)
- moved AVR_VDD 471.6 mm to (154.5, -23.5)
- moved CC8531_AVDD 471.6 mm to (154.5, -46.0)
- moved CC8531_IOVDD 471.6 mm to (154.5, -53.5)
- moved CODEC_AVDD 471.6 mm to (154.5, -61.0)
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Routing:
- net RED_BOT: track 0.00 -> 45.1 mm, vias 0 -> 1
- net BLUE_BOT: track 0.00 -> 44.4 mm, vias 0 -> 1
- net GREEN_BOT: track 0.00 -> 42.0 mm, vias 0 -> 1
- net RED_TOP: track 0.00 -> 40.8 mm, vias 0 -> 2
- net AUX_GREEN_TOP: track 0.99 -> 41.3 mm, vias 0 -> 1
- net AUX_BLUE_TOP: track 3.14 -> 43.1 mm, vias 0 -> 1
- net GREEN_TOP: track 0.00 -> 39.7 mm, vias 0 -> 1
- net AUX_RED_TOP: track 2.32 -> 39.5 mm, vias 0 -> 1
- net AUX_!CHANGE: track 17.5 -> 53.9 mm
- net AUX_SCLK: track 11.7 -> 47.8 mm
- net AUX_MISO: track 10.6 -> 46.5 mm
- net AUX_MOSI: track 9.96 -> 45.6 mm
- net BLUE_TOP: track 0.00 -> 35.3 mm, vias 0 -> 1
- net AUX_RED_BOT: track 0.07 -> 35.1 mm
- net AUX_CS: track 10.1 -> 44.8 mm
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- removed copper zone on layer 3, net 3.3V
- removed copper zone on layer 2, net AGND
- removed copper zone on layer 3, net AVDD
- removed copper zone on layer 3, net AVDD_CODEC
- removed copper zone on layer 3, net AVR_VDD
- removed copper zone on layer 3, net DVDD_CODEC
- removed copper zone on layer 2, net GND
- removed copper zone on layer 3, net IOVDD
