File: draft7.brd (EAGLE design)
At the start: 120 x 100 mm, 197 parts, among them Q1 Si2333, Q2 2N7002, Q3 2N7002, Q4 2N7002, Q5 2N7002, Q6 2N7002, Q7 2N7002, SW1 TOUCH_PAD-CIRCLE-15MM, SW10 TOUCH_PAD-CIRCLE-15MM, SW4 TOUCH_PAD-CIRCLE-15MM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

Commit message: Fixed stuff, created prototype board
Parts:
- added SJ1, SJ2, SJ3, SJ4: (no value), SparkFun-Passives (1):SJ_2S-NO
- EXT: value 0 -> (none); device rcl:R0603 -> SparkFun-Passives (1):SJ_2S-NO
- moved CC8531 14.5 mm to (48.8, 54.5)
- moved R5 12.0 mm to (49.0, 48.2)
- moved R17 6.05 mm to (29.0, 22.8), turned to 0 degrees
- moved L14 5.10 mm to (29.0, 20.8), turned to 180 degrees
- moved Q2 1.75 mm to (88.8, 3.50)
- moved Q3 1.75 mm to (88.8, 6.75)
- moved Q4 1.75 mm to (88.8, 10.0)
- moved Q5 1.75 mm to (101.0, 10.0)
- moved Q6 1.75 mm to (101.0, 6.75)
- moved Q7 1.75 mm to (101.0, 3.50)
- moved TO_MAIN2 1.75 mm to (95.0, 7.00)
- moved EXT 0.50 mm to (24.0, 88.2), turned to 90 degrees
- moved C45 0.25 mm to (40.0, 36.2)
Connections:
- new net M_BCLK: SJ1.2, U7.7
- new net M_DIN/S_DOUT: SJ4.2, U7.89
- new net M_DOUT/S_DIN: SJ3.2, U7.78
- new net M_WCLK: SJ2.2, U7.8
- new net S_BCLK: U7.90
- new net S_WCLK: U7.88
- net 3.3V: now also EXT.1; no longer EXT.2
- net BCLK: now also SJ1.1
- net DIN: now also SJ3.1
- net DOUT: now also SJ4.1
- net N$50: now also EXT.2; no longer EXT.1
- net WCLK: now also SJ2.1
Routing:
- net N$28: track 17.9 -> 3.06 mm
- net IOVDD: track 11.4 -> 17.5 mm, vias 8 -> 9
- net N$83: track 55.2 -> 51.7 mm
- net N$80: track 47.3 -> 44.7 mm
- net AUX_VDD: track 306.5 -> 304.0 mm
- net N$78: track 158.6 -> 156.9 mm
- net N$56: track 173.0 -> 171.2 mm
- net N$58: track 159.3 -> 157.5 mm
- net N$29: track 2.66 -> 4.00 mm
- net 3.3V: track 1.24 -> 2.29 mm
- net N$79: track 60.6 -> 59.6 mm
- net N$50: track 1.71 -> 2.44 mm

Commit message: New revision, changed proto board
Parts:
- removed R17: 0, rcl:R0603
- removed R27, R28, R29, R30: 0, 00-EvaLibrary:R0603
- removed SJ1, SJ3, SJ4: (no value), SparkFun-Passives (1):SJ_2S-NO
- added AGND, BCLK, DIN, DOUT, LINE_L, LINE_R, PHONE_L, PHONE_R: (no value), SparkFun-Passives (1):SJ_2S-NO
- added C70, C71: 0.47u, rcl:C0603
- moved C15 4.04 mm to (29.0, 57.2), turned to 0 degrees
- moved L3 3.75 mm to (27.5, 55.2)
- moved C1 2.80 mm to (28.8, 50.0), turned to 0 degrees
- moved L1 1.50 mm to (27.5, 52.0)
- moved R15 1.25 mm to (39.8, 21.8)
- renumbered SJ2 to WCLK
Connections:
- new net N$20: C70.2, R13.2
- new net N$24: C71.2, R16.2
- net AGND: now also AGND.2; no longer R17.2
- net BCLK: now also BCLK.1; no longer SJ1.1
- net DIN: now also DOUT.1; no longer SJ3.1
- net DOUT: now also DIN.1; no longer SJ4.1
- net GND: now also AGND.1; no longer R17.1
- net LINE_L: now also LINE_L.1; no longer R27.1
- net LINE_R: now also LINE_R.1; no longer R29.1
- net M_BCLK: now also BCLK.2; no longer SJ1.2
- net M_DIN/S_DOUT: now also DIN.2; no longer SJ4.2
- net M_DOUT/S_DIN: now also DOUT.2; no longer SJ3.2
- net N$43: now also C70.1, LINE_L.2, PHONE_L.2; no longer R13.2, R27.2, R28.2
- net N$45: now also C71.1, LINE_R.2, PHONE_R.2; no longer R16.2, R29.2, R30.2
- net PHONE_L: now also PHONE_L.1; no longer R28.1
- net PHONE_R: now also PHONE_R.1; no longer R30.1
Routing:
- net N$43: track 14.0 -> 3.90 mm
- net PHONE_L: track 6.34 -> 14.3 mm, vias 0 -> 2
- net GND: track 75.7 -> 78.4 mm
- net N$24: track 0.00 -> 2.62 mm
- net PHONE_R: track 12.5 -> 14.6 mm
- net LINE_R: track 8.09 -> 6.18 mm
- net LINE_L: track 15.1 -> 13.2 mm
- net N$45: track 3.41 -> 4.62 mm
- net N$54: track 5.02 -> 5.83 mm
- net N$40: track 21.2 -> 20.7 mm
- net AGND: vias 15 -> 14

Commit message: Switched to AT32UC3A3
Parts:
- added C72, C73, C75: 10p, 00-EvaLibrary:C0603
- added C74: 100n, 00-EvaLibrary:C0603
- added R17, R6: 39, rcl:R0603
- added R27: 6.8K, rcl:R0603
- added R28: 10K, rcl:R0603
- added RESET1: TACT_SWITCH-PTS-525, 00-EvaLibrary:PTS-525
- added U4: AT32UC3A3-LQFP-144, 00-EvaLibrary:LQFP-144
- added X2: 12MHz, 00-EvaLibrary:ABM8G
Connections:
- new net CTS: U4.123
- new net MISO0: U4.136
- new net MISO1: U4.114
- new net MOSI0: U4.138
- new net MOSI1: U4.128
- new net M_MCLK: U4.13
- new net N$39: R6.1, U4.8
- new net N$46: R17.1, U4.9
- new net N$47: C72.1, R27.2, U4.3
- new net N$52: C75.1, U4.18, X2.X1
- new net N$57: C73.1, U4.19, X2.X2
- new net RTS: U4.122
- new net RXD: U4.125
- new net SCLK0: U4.137
- new net SCLK1: U4.101
- new net TXD: U4.126
- net !RESET: now also C74.1, R28.1, RESET1.1, U4.106
- net AVR_PWR: now also R28.2
- net D+_UC: now also R17.2, U4.6
- net D-_UC: now also R6.2, U4.5
- net GND: now also C72.2, C73.2, C74.2, C75.2, R27.1, RESET1.3, X2.GND-1, X2.GND-2
- net M_BCLK: now also U4.38, U4.85
- net M_DIN/S_DOUT: now also U4.92
- net M_DOUT/S_DIN: now also U4.86
- net M_WCLK: now also U4.89
- net S_BCLK: now also U4.61, U4.91
- net S_WCLK: now also U4.44, U4.90
- net TCK: now also U4.107
- net TDI: now also U4.108
- net TDO: now also U4.105
- net TMS: now also U4.104
- net USBOTGID: now also U4.109
