File: draft7.sch (EAGLE design)
At the start: 183 parts, among them Q1 Si2333, Q2 2N7002, Q3 2N7002, Q4 2N7002, Q5 2N7002, Q6 2N7002, Q7 2N7002, SW1 TOUCH_PAD-CIRCLE-15MM, SW10 TOUCH_PAD-CIRCLE-15MM, SW4 TOUCH_PAD-CIRCLE-15MM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

Commit message: Fixed stuff, created prototype board
Parts:
- added SJ1, SJ2, SJ3, SJ4: SOLDERJUMPERNO, SparkFun-Passives (1):SOLDERJUMPERNO
- EXT: value 0 -> SOLDERJUMPERNO; device rcl:R-US_R0603 -> SparkFun-Passives (1):SOLDERJUMPERNO
Connections:
- removed net M_BLCK: U7A.PA14
- new net M_BCLK: SJ1.2, U7A.PA14
- net 3.3V: now also EXT.1; no longer EXT.2
- net BCLK: now also SJ1.1
- net DIN: now also SJ3.1
- net DOUT: now also SJ4.1
- net M_DIN/S_DOUT: now also SJ4.2
- net M_DOUT/S_DIN: now also SJ3.2
- net M_WCLK: now also SJ2.2
- net N$50: now also EXT.2; no longer EXT.1
- net WCLK: now also SJ2.1
Changed lines of the file:
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@@
 <part name="R17" library="rcl" deviceset="R-US_" device="R0603" value="0"/>
 <part name="GND12" library="SparkFun" deviceset="GND" device=""/>
-<part name="EXT" library="rcl" deviceset="R-US_" device="R0603" value="0"/>
 <part name="P+5" library="SparkFun" deviceset="3.3V" device=""/>
 <part name="U6" library="00-EvaLibrary" deviceset="LTC4088-1/2" device="" value="LTC4088-2"/>
@@
 <part name="R46" library="rcl" deviceset="R-US_" device="R0603" value="100K"/>
 <part name="GND55" library="SparkFun" deviceset="GND" device=""/>
+<part name="SJ1" library="SparkFun-Passives (1)" deviceset="SOLDERJUMPER" device="NO" value=""/>
+<part name="SJ2" library="SparkFun-Passives (1)" deviceset="SOLDERJUMPER" device="NO" value=""/>
+<part name="SJ3" library="SparkFun-Passives (1)" deviceset="SOLDERJUMPER" device="NO" value=""/>
+<part name="SJ4" library="SparkFun-Passives (1)" deviceset="SOLDERJUMPER" device="NO" value=""/>
+<part name="EXT" library="SparkFun-Passives (1)" deviceset="SOLDERJUMPER" device="NO" value=""/>
 </parts>
 <sheets>
@@
 <attribute name="VALUE" x="-224.79" y="-173.99" size="1.778" layer="96"/>
 </instance>
-<instance part="EXT" gate="G$1" x="-31.75" y="31.75" smashed="yes" rot="R180">
-<attribute name="NAME" x="-34.29" y="33.2486" size="1.778" layer="95"/>
-<attribute name="VALUE" x="-33.02" y="28.448" size="1.778" layer="96"/>
-</instance>
 <instance part="P+5" gate="G$1" x="-45.72" y="31.75" smashed="yes">
 <attribute name="VALUE" x="-46.736" y="35.306" size="1.778" layer="96"/>
@@
 <attribute name="VALUE" x="403.86" y="-472.44" size="1.778" layer="96"/>
 </instance>
+<instance part="SJ1" gate="1" x="251.46" y="-307.34"/>
+<instance part="SJ2" gate="1" x="251.46" y="-313.69"/>
+<instance part="SJ3" gate="1" x="251.46" y="-320.04"/>
+<instance part="SJ4" gate="1" x="251.46" y="-326.39"/>
+<instance part="EXT" gate="1" x="-31.75" y="31.75"/>
 </instances>
 <busses>
@@
 </segment>
 <segment>
-<pinref part="EXT" gate="G$1" pin="2"/>
 <pinref part="P+5" gate="G$1" pin="3.3V"/>
 <wire x1="-45.72" y1="31.75" x2="-36.83" y2="31.75" width="0.1524" layer="91"/>
+<pinref part="EXT" gate="1" pin="1"/>
 </segment>
 <segment>
@@
 <label x="-163.83" y="-88.9" size="1.778" layer="95" rot="R90" xref="yes"/>
 </segment>
+<segment>
+<pinref part="SJ1" gate="1" pin="1"/>
+<wire x1="246.38" y1="-307.34" x2="243.84" y2="-307.34" width="0.1524" layer="91"/>
+<label x="243.84" y="-307.34" size="1.778" layer="95" rot="R180" xref="yes"/>
+</segment>
 </net>
 <net name="WCLK" class="0">
@@
 <label x="-158.75" y="-88.9" size="1.778" layer="95" rot="R90" xref="yes"/>
 </segment>
+<segment>
+<pinref part="SJ2" gate="1" pin="1"/>
+<wire x1="246.38" y1="-313.69" x2="243.84" y2="-313.69" width="0.1524" layer="91"/>
+<label x="243.84" y="-313.69" size="1.778" layer="95" rot="R180" xref="yes"/>
+</segment>
 </net>
 <net name="RESET_CC8531" class="0">
@@
 <pinref part="L13" gate="G$1" pin="1"/>
 </segment>
+<segment>
+<pinref part="SJ3" gate="1" pin="1"/>
+<wire x1="246.38" y1="-320.04" x2="243.84" y2="-320.04" width="0.1524" layer="91"/>
+<label x="243.84" y="-320.04" size="1.778" layer="95" rot="R180" xref="yes"/>
+</segment>
 </net>
 <net name="DOUT" class="0">
@@
 <pinref part="L11" gate="G$1" pin="1"/>
 </segment>
+<segment>
+<pinref part="SJ4" gate="1" pin="1"/>
+<wire x1="246.38" y1="-326.39" x2="243.84" y2="-326.39" width="0.1524" layer="91"/>
+<label x="243.84" y="-326.39" size="1.778" layer="95" rot="R180" xref="yes"/>
+</segment>
 </net>
 <net name="REF" class="0">
@@
 <net name="N$50" class="0">
 <segment>
-<pinref part="EXT" gate="G$1" pin="1"/>
 <pinref part="CC_DEBUG" gate="G$1" pin="9"/>
 <wire x1="-26.67" y1="31.75" x2="-11.43" y2="31.75" width="0.1524" layer="91"/>
+<pinref part="EXT" gate="1" pin="2"/>
 </segment>
 </net>
@@
 </segment>
 </net>
-<net name="M_BLCK" class="0">
-<segment>
-<pinref part="U7" gate="A" pin="PA14"/>
-<wire x1="342.9" y1="-313.69" x2="337.82" y2="-313.69" width="0.1524" layer="91"/>
-<label x="337.82" y="-313.69" size="1.778" layer="95" rot="R180" xref="yes"/>
-</segment>
-</net>
 <net name="M_WCLK" class="0">
 <segment>
@@
 <label x="337.82" y="-318.77" size="1.778" layer="95" rot="R180" xref="yes"/>
 </segment>
+<segment>
+<pinref part="SJ2" gate="1" pin="2"/>
+<wire x1="256.54" y1="-313.69" x2="259.08" y2="-313.69" width="0.1524" layer="91"/>
+<label x="259.08" y="-313.69" size="1.778" layer="95" xref="yes"/>
+</segment>
 </net>
 <net name="M_DOUT/S_DIN" class="0">
@@
 <label x="337.82" y="-323.85" size="1.778" layer="95" rot="R180" xref="yes"/>
 </segment>
+<segment>
+<pinref part="SJ3" gate="1" pin="2"/>
+<wire x1="256.54" y1="-320.04" x2="259.08" y2="-320.04" width="0.1524" layer="91"/>
+<label x="259.08" y="-320.04" size="1.778" layer="95" xref="yes"/>
+</segment>
 </net>
 <net name="S_WCLK" class="0">
@@
 <label x="427.99" y="-334.01" size="1.778" layer="95" rot="R180" xref="yes"/>
 </segment>
+<segment>
+<pinref part="SJ4" gate="1" pin="2"/>
+<wire x1="256.54" y1="-326.39" x2="259.08" y2="-326.39" width="0.1524" layer="91"/>
+<label x="259.08" y="-326.39" size="1.778" layer="95" xref="yes"/>
+</segment>
 </net>
 <net name="S_BCLK" class="0">
@@
 </segment>
 </net>
+<net name="M_BCLK" class="0">
+<segment>
+<pinref part="SJ1" gate="1" pin="2"/>
+<wire x1="256.54" y1="-307.34" x2="259.08" y2="-307.34" width="0.1524" layer="91"/>
+<label x="259.08" y="-307.34" size="1.778" layer="95" xref="yes"/>
+</segment>
+<segment>
+<pinref part="U7" gate="A" pin="PA14"/>
+<wire x1="342.9" y1="-313.69" x2="337.82" y2="-313.69" width="0.1524" layer="91"/>
+<label x="337.82" y="-313.69" size="1.778" layer="95" rot="R180" xref="yes"/>
+</segment>
+</net>

Commit message: New revision, changed proto board
Parts:
- removed R17: 0, rcl:R-US_R0603
- removed R27, R28, R29, R30: 0, 00-EvaLibrary:R-US_R0603
- added AGND, LINE_L, LINE_R, PHONE_L, PHONE_R: SOLDERJUMPERNO, SparkFun-Passives (1):SOLDERJUMPERNO
- added C70, C71: 0.47u, rcl:C-EUC0603
- renumbered SJ1 to BCLK, SJ2 to WCLK, SJ3 to DOUT, SJ4 to DIN
Connections:
- new net N$20: C70.2, R13.2
- new net N$24: C71.2, R16.2
- net AGND: now also AGND.2; no longer R17.2
- net GND: now also AGND.1; no longer R17.1
- net LINE_L: now also LINE_L.1; no longer R27.1
- net LINE_R: now also LINE_R.1; no longer R29.1
- net N$43: now also C70.1, LINE_L.2, PHONE_L.2; no longer R13.2, R27.2, R28.2
- net N$45: now also C71.1, LINE_R.2, PHONE_R.2; no longer R16.2, R29.2, R30.2
- net PHONE_L: now also PHONE_L.1; no longer R28.1
- net PHONE_R: now also PHONE_R.1; no longer R30.1
Other:
- moved on the sheet: R13, R16

Commit message: Switched to AT32UC3A3
Parts:
- added C72, C73, C75: 10p, 00-EvaLibrary:C-EUC0603
- added C74: 100n, 00-EvaLibrary:C-EUC0603
- added R17, R6: 39, rcl:R-US_R0603
- added R27: 6.8K, rcl:R-US_R0603
- added R28: 10K, rcl:R-US_R0603
- added RESET1: TACT_SWITCH-PTS-525, 00-EvaLibrary:TACT_SWITCH-PTS-525
- added U4: AT32UC3A3-LQFP-144, 00-EvaLibrary:AT32UC3A3-LQFP-144
- added X2: 12MHz, 00-EvaLibrary:XTAL-ABRACONABM8G
Connections:
- new net CTS: U4A.PA01
- new net MISO0: U4A.PA11
- new net MISO1: U4A.PA19
- new net MOSI0: U4A.PA10
- new net MOSI1: U4A.PA16
- new net M_MCLK: U4C.PC04
- new net N$39: R6.1, U4M.D-_FS
- new net N$46: R17.1, U4M.D+_FS
- new net N$47: C72.1, R27.2, U4M.USB_VBIAS
- new net N$52: C75.1, U4C.PC02, X2.1
- new net N$57: C73.1, U4C.PC03, X2.2
- new net RTS: U4A.PA00
- new net RXD: U4A.PA03
- new net SCLK0: U4A.PA08
- new net SCLK1: U4A.PA15
- new net TXD: U4A.PA04
- net !RESET: now also C74.1, R28.1, RESET1.1, U4M.!RESET
- net AVR_PWR: now also R28.2
- net D+_UC: now also R17.2, U4M.D+_HS
- net D-_UC: now also R6.2, U4M.D-_HS
- net GND: now also C72.2, C73.2, C74.2, C75.2, R27.1, RESET1.3, X2.CASE
- net M_BCLK: now also U4X.PX23, U4X.PX35
- net M_DIN/S_DOUT: now also U4X.PX25
- net M_DOUT/S_DIN: now also U4X.PX24
- net M_WCLK: now also U4X.PX27
- net S_BCLK: now also U4X.PX28, U4X.PX34
- net S_WCLK: now also U4X.PX26, U4X.PX36
- net TCK: now also U4M.TCK
- net TDI: now also U4M.TDI
- net TDO: now also U4M.TDO
- net TMS: now also U4M.TMS
- net USBOTGID: now also U4A.PA21
