File: draft9.brd (EAGLE design)
At the start: 50 x 100 mm, 202 parts, among them Q1 Si2333, Q2 2N7002, Q3 2N7002, Q4 2N7002, Q5 2N7002, Q6 2N7002, Q7 2N7002, SW11 TOUCH_PAD-CIRCLE-15MM, SW2 TOUCH_PAD-CIRCLE-15MM, SW3 TOUCH_PAD-CIRCLE-15MM, SW4 TOUCH_PAD-CIRCLE-15MM, SW5 TOUCH_PAD-CIRCLE-15MM, SW6 TOUCH_PAD-CIRCLE-15MM, SW7 TOUCH_PAD-CIRCLE-15MM, U1 CC85XX, U11 CS4270-TSSOP24, U12 SN74LVC1G80DBV, U2 CC2591, U3 CS2300-MSOP10L, U4 AT32UC3A3-LQFP-144, U6 LTC4088-2, U8 AT42QT1110-TQFP, U9 LM4881, X1 48MHz, X2 12MHz

Commit message: Layout work
Parts:
- moved L5 212.8 mm to (45.0, 55.2), turned to 90 degrees
- moved R26 211.2 mm to (45.0, 48.8), turned to 90 degrees
- moved Q1 151.5 mm to (17.4, 83.3)
- moved C59 148.9 mm to (-140.5, 24.2)
- moved C61 148.9 mm to (-150.7, 24.2)
- moved C60 148.9 mm to (-145.6, 24.2)
- moved L13 133.0 mm to (49.0, 55.2), turned to 90 degrees
- moved L11 127.3 mm to (48.0, 52.0), turned to 90 degrees
- moved L9 118.4 mm to (47.0, 55.2), turned to 90 degrees
- moved L12 113.3 mm to (33.0, 60.5)
- moved C64 111.5 mm to (-60.4, -15.1)
- moved R11 110.5 mm to (41.8, 115.8)
- moved L6 110.3 mm to (46.0, 52.0), turned to 90 degrees
- moved R10 106.3 mm to (33.8, 66.0)
- moved L10 103.6 mm to (42.0, 84.5), turned to 180 degrees
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Connections:
- net !CS_CC8531: now also U4.133; no longer U4.127
- net !MUTE_L: now also U4.96; no longer U4.97
- net !MUTE_R: now also U4.95; no longer U4.96
- net !RESET_CC8531: now also U4.127; no longer U4.133
- net !RESET_CODEC: now also U4.97; no longer U4.95
Routing:
- net VBUS: track 0.00 -> 67.3 mm
- net D-_UC: track 8.06 -> 60.2 mm
- net D+_UC: track 7.85 -> 59.9 mm
- net SCLK1: track 2.00 -> 48.2 mm, vias 1 -> 3
- net MOSI1: track 0.00 -> 41.4 mm, vias 0 -> 3
- net MISO1: track 0.00 -> 32.4 mm, vias 0 -> 2
- net !PAIR: track 0.00 -> 28.5 mm, vias 0 -> 2
- net !RESET_CC8531: track 0.00 -> 28.2 mm, vias 0 -> 2
- net !CS_SD: track 0.00 -> 26.8 mm, vias 0 -> 2
- net UC_MCLK: track 0.00 -> 23.4 mm
- net DOUT: track 32.6 -> 55.6 mm, vias 2 -> 4
- net !CS_CC8531: track 0.00 -> 22.4 mm, vias 0 -> 2
- net !SD_CARD: track 0.00 -> 21.2 mm, vias 0 -> 2
- net MOSI0: track 22.4 -> 43.0 mm, vias 2 -> 4
- net WCLK: track 37.4 -> 57.5 mm
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
Commit message: More layout work
Parts:
- removed R11: 0, 00-EvaLibrary:R0603
- moved CC8531 161.4 mm to (48.8, 63.8), turned to 90 degrees
- moved L19 156.7 mm to (28.0, 13.5), turned to 90 degrees
- moved C21 147.8 mm to (41.2, 78.3)
- moved C22 147.5 mm to (35.0, 72.5), turned to 180 degrees
- moved C20 142.5 mm to (41.2, 80.2)
- moved C19 132.2 mm to (34.2, 70.0), turned to 270 degrees
- moved C76 130.7 mm to (38.8, 30.2), turned to 90 degrees
- moved C6 130.4 mm to (44.2, 58.0), turned to 270 degrees
- moved C18 129.2 mm to (36.2, 70.0), turned to 270 degrees
- moved AVR 128.8 mm to (1.25, 34.8), turned to 90 degrees
- moved C5 126.1 mm to (45.2, 63.0)
- moved C57 123.0 mm to (26.0, 13.5), turned to 90 degrees
- moved L20 120.5 mm to (16.8, 64.0), turned to 90 degrees
- moved CHARGE 118.9 mm to (1.50, 72.2), turned to 270 degrees
- moved R19 115.9 mm to (11.5, 73.2), turned to 90 degrees
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Connections:
- removed net 3.3V: L18.2, L19.2
- removed net AVDD_CODEC1: C14.1, C48.1, L21.1, U4.118
- removed net N$50: CC_DEBUG.9, R11.2
- net !CHANGE: now also U4.34; no longer U4.79
- net !CS_TOUCH: now also U4.33; no longer U4.80
- net AVDD_CODEC: now also C14.1, C48.1, L21.1, U4.118
- net D3.3V: now also L18.2, L19.2; no longer R11.1
Routing:
- net USBOTGID: track 0.00 -> 77.0 mm, vias 0 -> 2
- net SCLK0: track 29.9 -> 96.1 mm, vias 2 -> 4
- net MISO0: track 33.3 -> 98.6 mm, vias 0 -> 4
- net MOSI0: track 43.0 -> 104.1 mm, vias 4 -> 6
- net !CS_TOUCH: track 0.00 -> 56.3 mm, vias 0 -> 2
- net !CHANGE: track 0.00 -> 54.8 mm, vias 0 -> 2
- net BCLK: track 60.2 -> 100.5 mm
- net DGND: track 0.00 -> 35.8 mm, vias 0 -> 107
- net BAT: track 0.00 -> 34.0 mm, vias 0 -> 2
- net AVDD: track 0.00 -> 33.3 mm, vias 0 -> 13
- net VBUS: track 67.3 -> 97.7 mm, vias 0 -> 3
- net PA_EN: track 0.00 -> 27.0 mm, vias 0 -> 2
- net LNA_EN: track 0.00 -> 25.9 mm, vias 0 -> 2
- net N$28: track 0.00 -> 24.0 mm, vias 0 -> 2
- net N$32: track 0.00 -> 22.0 mm
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- added copper zone on layer 1, net AGND
- added copper zone on layer 16, net AGND
- added copper zone on layer 2, net AGND
- added copper zone on layer 3, net AVDD
- added copper zone on layer 3, net AVDD_CODEC
- added copper zone on layer 3, net AVR_VDD
- added copper zone on layer 2, net DGND
- added copper zone on layer 3, net DVDD_CODEC
- added copper zone on layer 3, net IOVDD

Commit message: Did a whole lot of things
Parts:
- removed C100, C101, C102: 100n, rcl:C0603
- removed C96: 1n, rcl:C0603
- removed C97: 1u, rcl:C0603
- removed L18: BEAD, SparkFun-Passives:0603
- removed MICROSD: MICROSD104031-0811, 00-EvaLibrary:MOLEX_104031-0811
- removed Q1: Si2333, SparkFun-DiscreteSemi:SOT23-3
- removed R23: 100K, rcl:R0603
- removed R44: 100, rcl:R0603
- removed RESET1: TACT_SWITCH-PTS-525, 00-EvaLibrary:PTS-525
- removed SW11, SW2, SW3, SW4, SW5, SW6, SW7: TOUCH_PAD-CIRCLE-15MM, 00-EvaLibrary:TOUCH-CIRCLE-15MM
- removed U12: SN74LVC1G80DBV, 00-EvaLibrary:SOT-23-5
- added AVR1: (no value), SparkFun-LED:LED-1206
- added BUTTON, NEXT, PLAY/PAUSE, PREV, STOP, VOL+, VOL-, WIRELESS: TOUCH_PAD-CIRCLE-10MM, 00-EvaLibrary:TOUCH-CIRCLE-10MM
- added C44, C46: 100n, 00-EvaLibrary:C0603
- added C47: 10u, 00-EvaLibrary:C0603
- added C55, C67, C68: 1u, 00-EvaLibrary:C0603
- added C56, C69: 1n, 00-EvaLibrary:C0603
- added C62: 2.2u, 00-EvaLibrary:C0603
- added C66: 220u, 00-EvaLibrary:C1210
- added GPIO, RESET: TACT_SWITCH-PTS-525, 00-EvaLibrary:PTS-525
- added L16: BEAD, SparkFun-Passives:0603
- added R11: 332, 00-EvaLibrary:R0603
- added R30, R32: 4.64K, 00-EvaLibrary:R0603
- added R38: 681, 00-EvaLibrary:R0603
- added R39: 4.53K, 00-EvaLibrary:R0603
- added R40, R41: 1K, 00-EvaLibrary:R0603
- added SD1: MICROSD104031-0811, 00-EvaLibrary:MOLEX_104031-0811
- added SERIAL: HEADER-6X1-961106-5500, 00-EvaLibrary:HEADER-3M-961-6P-2.54MM
- added U$6, U$7, U$8, U$9: (no value), 00-EvaLibrary:STANDOFF_3/16
- added U7: TLV700DDC, 00-EvaLibrary:SOT-23-5
- C1, C2: value 2.2u -> 100n; device rcl:C0603 -> 00-EvaLibrary:C0603
- C10: value 220p -> 1n; device rcl:C0603 -> 00-EvaLibrary:C0603
- C11, C15, C19, C31, C32, C40, C41, C42, C6, C64, C79: device rcl:C0603 -> 00-EvaLibrary:C0603
- C12, C7: value 100n -> 1n; device rcl:C0603 -> 00-EvaLibrary:C0603
- C13: value 2.2u -> 10p; device rcl:C0603 -> 00-EvaLibrary:C0603
- C14, C85, C95: value 1u -> 100n; device rcl:C0603 -> 00-EvaLibrary:C0603
- C16: value 10p -> 2.2u; device rcl:C0603 -> 00-EvaLibrary:C0603
- C17, C20, C86: value 1n -> 100n; device rcl:C0603 -> 00-EvaLibrary:C0603
- C18: value 10p -> 1u; device rcl:C0603 -> 00-EvaLibrary:C0603
- C21: value 18p -> 6.8p_HF; device rcl:C0603 -> 00-EvaLibrary:C0603
- C22: value 1n -> 100p_HF; device rcl:C0603 -> 00-EvaLibrary:C0603
- C23: value 1u -> 1.2p_HF; device rcl:C0603 -> 00-EvaLibrary:C0603
- C24: value 15p -> 1.8p_HF; device rcl:C0603 -> 00-EvaLibrary:C0603
- C25: value 6.8p_HF -> 1u; device rcl:C0603 -> 00-EvaLibrary:C0603
- C26: value 100p_HF -> 27p; device rcl:C0603 -> 00-EvaLibrary:C0603
- C27: value 1.2p_HF -> 27p; device rcl:C0603 -> 00-EvaLibrary:C0603
- C28: value 1.8p_HF -> 1u; device rcl:C0603 -> 00-EvaLibrary:C0603
- C29: value 15p -> 100n; device rcl:C0603 -> 00-EvaLibrary:C0603
- C3: value 1u -> 2.2u; device rcl:C0603 -> 00-EvaLibrary:C0603
- C30: value 10n -> 100n; device rcl:C0603 -> 00-EvaLibrary:C0603
- C33, C49: value 1u -> 1n; device rcl:C0603 -> 00-EvaLibrary:C0603
- C34, C48, C63, C77: value 100n -> 1u; device rcl:C0603 -> 00-EvaLibrary:C0603
- C35, C43, C58: value 10n -> 1n; device rcl:C0603 -> 00-EvaLibrary:C0603
- C36: value 220u -> 470n; device 00-EvaLibrary:C1210 -> 00-EvaLibrary:C0603
- C37, C54: value 100n -> 2.2u
- C38: value 100n -> 470n; device rcl:C0603 -> 00-EvaLibrary:C0603
- C39: value 220u -> 100n; device 00-EvaLibrary:C1210 -> 00-EvaLibrary:C0603
- C4: value 100n -> 100n_HF; device rcl:C0603 -> 00-EvaLibrary:C0603
- C45: value 1n -> 10u; device rcl:C0603 -> 00-EvaLibrary:C0603
- C5: value 100n -> 220p_HF; device rcl:C0603 -> 00-EvaLibrary:C0603
- C50: value 1n -> 1u; device rcl:C0603 -> 00-EvaLibrary:C0603
- C51: value 10u -> 1n
- C52, C80: value 10u -> 1u; device rcl:C0603 -> 00-EvaLibrary:C0603
- C53: value 10u -> 220u; device rcl:C0603 -> 00-EvaLibrary:C1210
- C57, C65: value 2.2u -> 1u; device rcl:C0603 -> 00-EvaLibrary:C0603
- C59, C60, C61: value 10n -> 10u; device rcl:C0603 -> 00-EvaLibrary:C0603
- C70: value 470n -> 10u
- C71: value 470n -> 1u; device rcl:C0603 -> 00-EvaLibrary:C0603
- C72: value 10p -> 1u
- C73: value 10p -> 100n
- C74: value 100n -> 1u
- C75: value 10p -> 1n
- C76: value 10u -> 10p; device rcl:C0603 -> 00-EvaLibrary:C0603
- C78: value 10u -> 1n; device rcl:C0603 -> 00-EvaLibrary:C0603
- C8: value 100n -> 10p; device rcl:C0603 -> 00-EvaLibrary:C0603
- C81, C82: value 470n -> 100n; device rcl:C0603 -> 00-EvaLibrary:C0603
- C83: value 1u -> 10p; device rcl:C0603 -> 00-EvaLibrary:C0603
- C84: value 1n -> 10p; device rcl:C0603 -> 00-EvaLibrary:C0603
- C87, C89, C91, C93: value 1u -> 10n; device rcl:C0603 -> 00-EvaLibrary:C0603
- C88, C90, C92, C94: value 1n -> 10n; device rcl:C0603 -> 00-EvaLibrary:C0603
- C9: value 100n -> 18p; device rcl:C0603 -> 00-EvaLibrary:C0603
- C98: value 1n -> 470n; device rcl:C0603 -> 00-EvaLibrary:C0603
- C99: value 1u -> 470n; device rcl:C0603 -> 00-EvaLibrary:C0603
- L1, L2: value BEAD -> BEAD_HF; device SparkFun-Passives:0603 -> 00-EvaLibrary:0603
- L10: value 1.5n_HF -> 6.8n; device SparkFun-Passives:0603 -> 00-EvaLibrary:0603
- L11, L13, L14, L19, L20, L21, L3, L9: device SparkFun-Passives:0603 -> 00-EvaLibrary:0603
- L17: value 3.3u -> BEAD; device 00-EvaLibrary:IFSC-1111AB-01 -> 00-EvaLibrary:0603
- L4: value 6.8n -> 2.2n_HF; device SparkFun-Passives:0603 -> 00-EvaLibrary:0603
- L5: value 6.8n -> 3.9n_HF; device SparkFun-Passives:0603 -> 00-EvaLibrary:0603
- L6: value 6.8n -> 1.5n_HF; device SparkFun-Passives:0603 -> 00-EvaLibrary:0603
- L7: value 2.2n_HF -> 6.8n; device SparkFun-Passives:0603 -> 00-EvaLibrary:0603
- L8: value 3.9n_HF -> 6.8n; device SparkFun-Passives:0603 -> 00-EvaLibrary:0603
- R1, R2: value 0 -> 4.32K
- R12: value 20K -> 100
- R13, R16: value 20K -> 1M
- R14: value 4.7K -> 20K; device rcl:R0603 -> 00-EvaLibrary:R0603
- R15: value 20K -> 39
- R17, R25, R5: device rcl:R0603 -> 00-EvaLibrary:R0603
- R18: value 330 -> 10K
- R19: value 8.2 -> 100K
- R20: value 2.94K -> 100K
- R21: value 1K -> 20K
- R22: value 1M -> 100K; device rcl:R0603 -> 00-EvaLibrary:R0603
- R24: value 1M -> 0; device rcl:R0603 -> 00-EvaLibrary:R0603
- R27: value 6.8K -> 6.81K; device rcl:R0603 -> 00-EvaLibrary:R0603
- R28: value 4.7K -> 100K; device rcl:R0603 -> 00-EvaLibrary:R0603
- R29, R33, R34, R35: value 4.7K -> 4.64K; device rcl:R0603 -> 00-EvaLibrary:R0603
- R3: value 100 -> 56.2K; device rcl:R0603 -> 00-EvaLibrary:R0603
- R31: value 10K -> 4.64K; device rcl:R0603 -> 00-EvaLibrary:R0603
- R36: value 100K -> 4.64K; device rcl:R0603 -> 00-EvaLibrary:R0603
- R37: value 4.7K -> 10K; device rcl:R0603 -> 00-EvaLibrary:R0603
- R4: value 56k -> 100; device rcl:R0603 -> 00-EvaLibrary:R0603
- R6: value 39 -> 10K; device rcl:R0603 -> 00-EvaLibrary:R0603
- R7: value 10K -> 20K; device rcl:R0603 -> 00-EvaLibrary:R0603
- R8: value 4.3K -> 100; device rcl:R0603 -> 00-EvaLibrary:R0603
- R9: value 4.3K -> 20K; device rcl:R0603 -> 00-EvaLibrary:R0603
- U1: value CC85XX -> CC2591; device 00-EvaLibrary:S-PVQFN-N40 -> 00-EvaLibrary:S-PVQFN-N16
- U10: value (none) -> AT32UC3A3-LQFP-144; device 00-EvaLibrary:SOT-223 -> 00-EvaLibrary:LQFP-144
- U11: value CS4270-TSSOP24 -> AT42QT1110-QFN-32; device 00-EvaLibrary:TSSOP-24L -> 00-EvaLibrary:QFN-32
- U2: value CC2591 -> CC85XX; device 00-EvaLibrary:S-PVQFN-N16 -> 00-EvaLibrary:S-PVQFN-N40
- U3: value CS2300-MSOP10L -> CS4270-TSSOP24; device 00-EvaLibrary:MSOP-10L -> 00-EvaLibrary:TSSOP-24L
- U4: value AT32UC3A3-LQFP-144 -> LM4881; device 00-EvaLibrary:LQFP-144 -> 00-EvaLibrary:SO08
- U6: value LTC4088-2 -> BQ2409XDGQ; device 00-EvaLibrary:DFN-14 -> 00-EvaLibrary:S-PDSO-G10
- U8: value AT42QT1110-TQFP -> SN74LVC1G80DBV; device 00-EvaLibrary:S-PQFP-N32 -> 00-EvaLibrary:SOT-23-5
- U9: value LM4881 -> CS2300-MSOP10L; device 00-EvaLibrary:SO08 -> 00-EvaLibrary:MSOP-10L
- moved R29 264.1 mm to (78.5, 99.0), flipped to the bottom, turned to 180 degrees
- moved LED_UR 241.1 mm to (95.5, 90.2), flipped to the bottom, turned to 180 degrees
- moved R28 228.9 mm to (65.5, 98.8), flipped to the bottom
- moved TO_MAIN1 225.4 mm to (86.0, 96.0), flipped to the bottom, turned to 180 degrees
- moved R35 213.7 mm to (61.0, 93.2), flipped to the bottom, turned to 90 degrees
- moved R33 211.9 mm to (74.0, 87.5), flipped to the bottom, turned to 180 degrees
- moved R34 209.2 mm to (64.2, 88.8), flipped to the bottom
- moved LED_LR 200.9 mm to (95.5, 9.75), flipped to the bottom
- moved Q7 199.9 mm to (80.8, 3.00), flipped to the bottom, turned to 90 degrees
- moved U8 194.9 mm to (40.0, 44.5), turned to 180 degrees
- moved Q5 192.7 mm to (80.8, 6.25), flipped to the bottom, turned to 90 degrees
- moved LED_UL 192.5 mm to (54.5, 90.2), flipped to the bottom
- moved C30 188.0 mm to (45.2, 24.8), turned to 270 degrees
- moved LED_LL 185.7 mm to (54.5, 9.75), flipped to the bottom, turned to 180 degrees
- moved Q3 185.6 mm to (80.8, 9.50), flipped to the bottom, turned to 90 degrees
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- renumbered CC8531 to CC1, USB2 to USB
Connections:
- removed net !AVR_LED: AVR.C, U4.50
- removed net !CS_SD: MICROSD.CD/DAT3, U4.17
- removed net N$36: L17.1, U6.12
- removed net N$37: R21.2, U6.5, U6.6
- removed net N$38: R19.2, R20.2, U6.2
- removed net N$48: C54.1, R19.1
- new net !AVR_LED0: AVR.C, U10.50
- new net !AVR_LED1: AVR1.C, U10.40
- new net !GPIO: GPIO.2, U10.74
- new net AUX_VDD2: LED_LL.2, LED_LL.2-2, LED_LR.2, LED_LR.2-2, LED_UL.2, LED_UL.2-2, LED_UR.2, LED_UR.2-2, TO_MAIN2.1, TO_MAIN2.2
- new net AUX_VSS1: Q2.2, Q3.2, Q4.2, Q5.2, Q6.2, Q7.2, TO_MAIN2.10, TO_MAIN2.9
- new net MCI-CLK: SD1.CLK, U10.26
- new net MCI-CMD: R22.1, SD1.CMD, U10.28
- new net MCI-DATA0: R20.1, SD1.DAT0, U10.23
- new net MCI-DATA1: SD1.DAT1, U10.14
- new net MCI-DATA2: SD1.DAT2, U10.29
- new net MCI-DATA3: SD1.CD/DAT3, U10.30
- new net N$11: PLAY/PAUSE.P$1, R36.2
- new net N$17: C94.1, U11.23
- new net N$44: R38.2, U6.2
- new net N$50: F1.2, L21.2, U5.1
- new net N$6: C94.2, R36.1, U11.22
- new net N$66: R37.2, U6.9
- new net N$69: R39.2, U6.4
- net !CHANGE: now also TO_AUX2.9, U10.34; no longer TO_AUX1.9, U4.34
- net !CS_CC8531: now also U10.133, U2.3; no longer U1.3, U4.133
- net !CS_CLOCK: now also U10.100, U9.8; no longer U3.8, U4.46
- net !CS_CODEC: now also U10.93, U3.11; no longer U11.11, U4.94
- net !CS_TOUCH: now also TO_AUX2.7, U10.51; no longer TO_AUX1.7, U4.33
- net !MUTE_L: now also U10.96, U3.21; no longer U11.21, U4.96
- net !MUTE_R: now also U10.95, U3.24; no longer U11.24, U4.95
- net !PAIR: now also U10.129, U2.7; no longer U1.7, U4.129
- net !RESET: now also C73.1, R18.1, RESET.1, U10.106; no longer C74.1, R7.1, RESET1.1, U4.106
- net !RESET_CC8531: now also L7.2, U10.127; no longer L4.2, U4.127
- net !RESET_CODEC: now also U10.97, U3.14; no longer U11.14, U4.97
- net !SD_CARD: now also SD1.SWB, U10.27; no longer MICROSD.SWA, U4.14
- net A3.3V: now also C70.1, L15.2, L20.2, U7.5; no longer C76.1, L14.2, L21.2, U10.3
- net AGND: now also C30.2, C39.2, C44.2, C45.2, C46.2, C47.2, C63.2, C64.2, C65.2, C70.2, C71.2, C98.2, C99.2, R19.1, R24.2, U10.117, U3.20, U4.2, U7.2; no longer C14.2, C33.2, C34.2, C38.2, C48.2, C76.2, C77.2, C78.2, C79.2, C80.2, R1.2, R23.1, U10.2, U10.4, U11.20, U4.117, U9.2
- net ALL_GND: now also C59.2, C60.2, R24.1, R26.1, R37.1, R38.1, R39.1, U6.3, U6.7; no longer C51.2, C52.2, C54.2, R1.1, R2.1, R20.1, R21.1, U6.1, U6.14, U6.4
- net AUDIO: now also C53.1, R7.1, U10.116, U4.7; no longer C36.1, R12.1, U4.116, U9.7
- net AUX_!CHANGE: now also U11.28; no longer U8.28
- net AUX_BLUE_TOP: now also Q6.1; no longer Q4.1
- net AUX_CS: now also U11.14; no longer U8.14
- net AUX_GREEN_BOT: now also Q5.1; no longer Q6.1
- net AUX_GREEN_TOP: now also Q4.1; no longer Q3.1
- net AUX_MISO: now also U11.16; no longer U8.16
- net AUX_MOSI: now also U11.15; no longer U8.15
- net AUX_RED_BOT: now also Q3.1; no longer Q5.1
- net AUX_SCLK: now also U11.17; no longer U8.17
- net AUX_VDD: now also C85.1, C86.1, R28.2, U11.18, U11.4; no longer C63.1, C64.1, LED_LL.2, LED_LL.2-2, LED_LR.2, LED_LR.2-2, LED_UL.2, LED_UL.2-2, LED_UR.2, LED_UR.2-2, R36.2, TO_MAIN2.1, TO_MAIN2.2, U8.18, U8.4
- net AUX_VSS: now also C85.2, C86.2, U11.21, U11.5, U11.GND; no longer C63.2, C64.2, Q2.2, Q3.2, Q4.2, Q5.2, Q6.2, Q7.2, TO_MAIN2.10, TO_MAIN2.9, U8.21, U8.5
- net AVDD: now also C1.1, C13.1, C14.1, C3.1, C4.1, C5.1, C7.1, L1.1, R1.2, U1.1, U1.10, U1.13, U1.16, U2.20, U2.23, U2.26, U2.27, U2.28, U2.31; no longer C11.1, C16.1, C17.1, C18.1, C2.1, C21.1, C22.1, L3.1, R9.2, U1.20, U1.23, U1.26, U1.27, U1.28, U1.31, U2.1, U2.10, U2.13, U2.16
- net AVDD_CODEC: now also C30.1, C39.1, C64.1, C65.1, L15.1, L20.1, R10.2, R13.2, R16.2, U10.118, U3.19, U4.6; no longer C14.1, C34.1, C38.1, C48.1, L14.1, L21.1, R22.2, R24.2, R31.2, U11.19, U4.118, U9.6
- net AVR_VDD: now also C32.1, C33.1, C34.1, C35.1, C37.1, C42.1, C43.1, C48.1, C51.1, C55.1, C56.1, C57.1, C58.1, C72.1, C74.1, C75.1, C77.1, C78.1, L16.1, R18.2, R20.2, R22.2, R5.2, R8.2, SD1.VDD, U10.10, U10.103, U10.130, U10.142, U10.143, U10.2, U10.21, U10.48, U10.64, U10.81; no longer C100.1, C102.1, C13.1, C83.1, C84.1, C85.1, C86.1, C87.1, C88.1, C89.1, C90.1, C91.1, C92.1, C93.1, C94.1, C96.1, C97.1, C98.1, C99.1, L20.1, MICROSD.VDD, R44.2, R7.2, U12.5, U3.1, U4.10, U4.103, U4.130, U4.142, U4.143, U4.2, U4.21, U4.48, U4.64, U4.81
- net BAT: now also C60.1, F1.1, R11.2, U2.29, U6.10; no longer Q1.2, U1.29, U6.9
- net BCLK: now also L9.1, U10.38, U10.61, U10.85, U10.91, U3.4; no longer L6.1, U11.4, U4.38, U4.61, U4.85, U4.91
- net BLUE_BOT: now also TO_AUX1.8, U10.84; no longer TO_AUX2.8, U4.84
- net BLUE_TOP: now also TO_AUX1.3, U10.68; no longer TO_AUX2.3, U4.68
- net CTS: now also SERIAL.5, U10.62; no longer U4.62
- net D+_UC: now also R15.2, U10.6; no longer R17.2, U4.6
- net D-_UC: now also R17.2, U10.5; no longer R6.2, U4.5
- net D3.3V: now also C61.1, C79.1, C80.1, C81.1, L14.2, L16.2, L17.2, R12.2, U8.5, U9.1; no longer C53.1, L15.2, L18.2, L20.2, R3.2
- net DAC0_N: now also U10.126; no longer U4.126
- net DAC0_P: now also U10.125; no longer U4.125
- net DAC1_N: now also U10.112; no longer U4.112
- net DAC1_P: now also U10.111; no longer U4.111
- net DGND: now also C14.2, C25.2, C26.2, C33.2, C34.2, C35.2, C43.2, C48.2, C51.2, C54.2, C55.2, C56.2, C58.2, C61.2, C62.2, C68.2, C69.2, C76.2, C77.2, C78.2, C79.2, C80.2, C81.2, C82.2, GPIO.4, L6.1, R2.1, R26.2, R3.1, R6.1, RESET.3, SD1.GND1, SD1.GND2, SD1.GND3, SD1.GND4, SD1.SWA, SD1.VSS, SERIAL.6, TO_AUX1.9, TO_AUX2.6, TO_AUX2.8, U1.12, U1.14, U1.8, U1.9, U10.102, U10.131, U10.140, U10.144, U10.20, U10.4, U10.47, U10.65, U10.7, U10.82, U2.19, U2.32, U2.33, U2.34, U2.35, U3.6, U8.3, U9.2, U9.7; no longer C100.2, C101.2, C102.2, C21.2, C22.2, C45.2, C53.2, C65.2, C85.2, C86.2, C87.2, C88.2, C89.2, C90.2, C91.2, C92.2, C93.2, C94.2, C96.2, C97.2, C98.2, C99.2, L10.1, MICROSD.GND1, MICROSD.GND2, MICROSD.GND3, MICROSD.GND4, MICROSD.SWB, MICROSD.VSS, R10.1, R2.2, R4.1, R8.1, RESET1.3, TO_AUX1.6, TO_AUX1.8, TO_AUX2.9, U11.6, U12.3, U2.12, U2.14, U2.8, U2.9, U3.2, U3.7, U4.102, U4.131, U4.140, U4.144, U4.20, U4.4, U4.47, U4.65, U4.7, U4.82
- net DIN: now also U10.86, U3.1; no longer U11.1, U4.86
- net DOUT: now also U10.92, U3.7; no longer U11.7, U4.92
- net DVDD_CODEC: now also C28.1, C29.1, L14.1, U3.5, U3.8; no longer C32.1, C37.1, L15.1, U11.5, U11.8
- net GREEN_BOT: now also TO_AUX1.6, U10.139; no longer TO_AUX2.6, U4.139
- net GREEN_TOP: now also TO_AUX1.5, U10.75; no longer TO_AUX2.5, U4.75
- net IN_L: now also C38.1, R19.2; no longer C82.1, R23.2
- net IN_R: now also C36.1; no longer C81.1
- net IOVDD: now also C11.1, C16.1, C17.1, C18.1, C2.1, L3.1, U2.10, U2.12, U2.18, U2.37, U2.40; no longer C1.1, C3.1, C4.1, C5.1, C7.1, L1.1, U1.10, U1.12, U1.18, U1.37, U1.40
- net LINEIN_SENSE: now also R13.1, U10.114; no longer R22.1, U4.114
- net LNA_EN: now also U1.6, U2.38; no longer U1.38, U2.6
- net MCLK: now also L8.1, U8.2, U9.3; no longer R26.1, U11.3, U12.2
- net MISO0: now also U10.136, U2.6, U3.9; no longer TO_AUX1.3, U1.6, U11.9, U4.136
- net MISO1: now also TO_AUX2.3, U10.11; no longer MICROSD.DAT0, U4.11
- net MOSI0: now also U10.138, U2.5, U3.12, U9.10; no longer TO_AUX1.5, U1.5, U11.12, U4.138
- net MOSI1: now also TO_AUX2.5, U10.16; no longer MICROSD.CMD, U3.10, U4.16
- net N$1: now also C26.1, U2.21; no longer C29.1, U1.21
- net N$10: now also AVR1.A, R5.1; no longer L5.1, R26.2
- net N$12: now also R8.1; no longer R44.1
- net N$14: now also C23.1, L4.2, L5.1; no longer C27.1, L7.2, L8.1
- net N$15: now also C21.1, L5.2; no longer C25.1, L8.2
- net N$16: now also C21.2, C22.1, C24.1, L6.2; no longer C25.2, C26.1, C28.1, L10.2
- net N$18: now also U2.36; no longer U1.36
- net N$19: now also R3.2, U2.30; no longer R4.2, U1.30
- net N$2: now also C27.1, U2.22; no longer C24.1, U1.22
- net N$20: now also C52.2, C98.1, R9.2; no longer C70.2, R13.2
- net N$21: now also C25.1, U2.39; no longer C23.1, U1.39
- net N$22: now also C71.1, L21.1, U7.1, U7.3; no longer F1.2, U10.1, U5.1
- net N$23: now also L8.2, U2.13; no longer L5.2, U1.13
- net N$24: now also C67.2, C99.1, R14.2; no longer C71.2, R16.2
- net N$25: now also L10.2, U2.15; no longer L9.2, U1.15
- net N$26: now also C63.1, U4.1; no longer C33.1, U9.1
- net N$27: now also U2.17; no longer U1.17
- net N$28: now also R4.1, U2.9; no longer R5.1, U1.9
- net N$29: now also R4.2; no longer R5.2
- net N$30: now also C90.2, R32.1, U11.9; no longer C58.2, R33.1, U8.9
- net N$31: now also R12.1; no longer R3.1
- net N$32: now also U6.8; no longer U6.7
- net N$33: now also R11.1; no longer R18.1
- net N$34: now also C68.1, C69.1, U10.141; no longer C42.1, C45.1, U4.141
- net N$35: now also U10.45, U9.5; no longer U3.5, U4.45
- net N$39: now also R17.1, U10.8; no longer R6.1, U4.8
- net N$4: now also U2.16; no longer U1.16
- net N$40: now also C66.1, R21.1, U4.5; no longer C39.1, R15.1, U9.5
- net N$41: now also C91.2, R33.1, U11.11; no longer C59.2, R34.1, U8.11
- net N$42: now also C92.2, R34.1, U11.13; no longer C60.2, R35.1, U8.13
- net N$43: now also C87.2, R29.1, U11.1; no longer C30.2, R14.1, U8.1
- net N$45: now also C88.2, R30.1, U11.3; no longer C35.2, R28.1, U8.3
- net N$46: now also R15.1, U10.9; no longer R17.1, U4.9
- net N$47: now also C76.1, U10.3; no longer C72.1, U4.3
- net N$49: now also C67.1, R40.1; no longer C52.1, F1.1, L17.2, Q1.3, U6.10, U6.3
- net N$5: now also L9.2, U2.14; no longer L6.2, U1.14
- net N$51: now also C52.1, R41.1; no longer Q1.1, U6.8
- net N$52: now also C83.1, U10.18; no longer C75.1, U4.18
- net N$53: now also R7.2, R9.1, U4.8; no longer R12.2, R13.1, U9.8
- net N$54: now also R14.1, R21.2, U4.4; no longer R15.2, R16.1, U9.4
- net N$55: now also R10.1, U4.3; no longer R31.1, U9.3
- net N$57: now also C84.1, U10.19; no longer C73.1, U4.19
- net N$58: now also Q4.3; no longer Q3.3
- net N$59: now also C87.1, U11.32; no longer C30.1, U8.32
- net N$60: now also C90.1, U11.8; no longer C58.1, U8.8
- net N$61: now also R32.2, VOL+.P$1; no longer R33.2, SW4.P$1
- net N$62: now also C91.1, U11.10; no longer C59.1, U8.10
- net N$63: now also R33.2, WIRELESS.P$1; no longer R34.2, SW5.P$1
- net N$64: now also C92.1, U11.12; no longer C60.1, U8.12
- net N$65: now also R34.2, VOL-.P$1; no longer R35.2, SW6.P$1
- net N$67: now also C54.1, L17.1, TO_AUX1.1, TO_AUX1.2; no longer C57.1, L19.1, TO_AUX2.1, TO_AUX2.2
- net N$7: now also R2.2, U1.15; no longer R8.2, U2.15
- net N$71: now also C93.2, R35.1, U11.19; no longer C61.2, R37.1, U8.19
- net N$72: now also PREV.P$1, R35.2; no longer R37.2, SW7.P$1
- net N$76: now also C93.1, U11.20; no longer C61.1, U8.20
- net N$77: now also R28.1, U11.29; no longer R36.1, U8.29
- net N$78: now also Q6.3; no longer Q4.3
- net N$79: now also Q3.3; no longer Q5.3
- net N$8: now also R1.1, U1.7; no longer R9.1, U2.7
- net N$80: now also Q5.3; no longer Q6.3
- net N$84: now also C62.1, L19.1, TO_AUX2.2, TO_AUX2.4; no longer C65.1, L18.1, TO_AUX1.2, TO_AUX1.4
- net N$85: now also R29.2, STOP.P$1; no longer R14.2, SW2.P$1
- net N$86: now also C88.1, U11.2; no longer C35.1, U8.2
- net N$87: now also NEXT.P$1, R30.2; no longer R28.2, SW3.P$1
- net N$88: now also C46.1, C47.1, U3.17; no longer C77.1, C78.1, U11.17
- net N$89: now also C44.1, C45.1, U3.18; no longer C79.1, C80.1, U11.18
- net N$9: now also C22.2; no longer C26.2
- net N$90: now also C89.2, R31.1, U11.6; no longer C43.2, R29.1, U8.6
- net N$91: now also C36.2, U3.15; no longer C81.2, U11.15
- net N$92: now also C38.2, U3.16; no longer C82.2, U11.16
- net N$93: now also C89.1, U11.7; no longer C43.1, U8.7
- net N$94: now also C82.1, U9.6; no longer C101.1, U3.6
- net N$95: now also BUTTON.P$1, R31.2; no longer R29.2, SW11.P$1
- net OUT_L: now also R41.2, U3.23; no longer C70.1, U11.23
- net OUT_R: now also R40.2, U3.22; no longer C71.1, U11.22
- net PA_EN: now also R6.2, U1.5; no longer R10.2, U2.5
- net PHONE_L: now also C53.2; no longer C36.2
- net PHONE_R: now also C66.2; no longer C39.2
- net PHONE_SENSE: now also R16.1, U10.115; no longer R24.1, U4.115
- net RED_BOT: now also TO_AUX1.4, U10.132; no longer TO_AUX2.4, U4.132
- net RED_TOP: now also TO_AUX1.7, U10.83; no longer TO_AUX2.7, U4.83
- net RF_N: now also U1.2, U2.25; no longer U1.25, U2.2
- net RF_P: now also U1.4, U2.24; no longer U1.24, U2.4
- net RTS: now also SERIAL.1, U10.63; no longer U4.63
- net RXD: now also SERIAL.3, U10.55; no longer U4.55
- net SCLK0: now also U10.137, U2.4, U3.10, U9.9; no longer TO_AUX1.1, U1.4, U11.10, U4.137
- net SCLK1: now also TO_AUX2.1, U10.135; no longer MICROSD.CLK, U3.9, U4.135
- net TCK: now also U10.107; no longer U4.107
- net TDI: now also U10.108; no longer U4.108
- net TDO: now also U10.105; no longer U4.105
- net TMS: now also U10.104; no longer U4.104
- net TXD: now also SERIAL.2, U10.59; no longer U4.59
- net UC_MCLK: now also U10.13, U8.1, U8.4; no longer U12.1, U12.4, U4.13
- net USBOTGID: now also U10.121; no longer U4.121
- net VBUS: now also C59.1, U10.1, U6.1; no longer C51.1, R18.2, U4.1, U6.11, U6.13
- net WCLK: now also L10.1, U10.44, U10.89, U10.90, U3.2; no longer L9.1, U11.2, U4.44, U4.89, U4.90
Routing:
- net AUX_VDD2: track 0.00 -> 242.9 mm, vias 0 -> 5
- net N$56: track 0.00 -> 216.5 mm
- net N$58: track 0.00 -> 215.9 mm, vias 0 -> 2
- net N$78: track 0.00 -> 211.5 mm, vias 0 -> 4
- net N$50: track 0.00 -> 139.2 mm, vias 0 -> 2
- net N$95: track 0.00 -> 77.0 mm, vias 0 -> 1
- net N$63: track 0.00 -> 74.0 mm, vias 0 -> 1
- net N$65: track 0.00 -> 60.9 mm, vias 0 -> 1
- net N$79: track 0.00 -> 60.2 mm, vias 0 -> 3
- net N$61: track 0.00 -> 54.1 mm, vias 0 -> 1
- net N$83: track 0.00 -> 50.3 mm, vias 0 -> 2
- net BAT: track 34.0 -> 84.0 mm, vias 2 -> 5
- net N$35: track 9.49 -> 55.4 mm, vias 0 -> 2
- net MISO0: track 98.6 -> 52.8 mm, vias 4 -> 2
- net N$80: track 0.00 -> 45.3 mm, vias 0 -> 2
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- added copper zone on layer 1, net ALL_GND
- added copper zone on layer 2, net ALL_GND
- added copper zone on layer 16, net AUX_VSS
- added copper zone on layer 3, net D3.3V
- added copper zone on layer 1, net DGND
Other:
- board size 50 x 100 mm -> 100 x 100 mm

Commit message: Minor revisions
Parts:
- moved BUTTON 5.00 mm to (92.5, 20.0)
- moved C85 5.00 mm to (80.2, 95.0)
- moved C86 5.00 mm to (68.0, 90.8)
- moved C87 5.00 mm to (80.2, 99.0)
- moved C88 5.00 mm to (80.2, 97.0)
- moved C89 5.00 mm to (79.8, 92.0)
- moved C90 5.00 mm to (79.0, 89.5)
- moved C91 5.00 mm to (75.8, 88.8)
- moved C92 5.00 mm to (72.5, 88.8)
- moved C93 5.00 mm to (68.0, 93.2)
- moved C94 5.00 mm to (68.0, 97.2)
- moved LED_LL 5.00 mm to (59.5, 9.75)
- moved LED_LR 5.00 mm to (100.5, 9.75)
- moved LED_UL 5.00 mm to (59.5, 90.2)
- moved LED_UR 5.00 mm to (100.5, 90.2)
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Connections:
- net BCLK: no longer U10.38
Routing:
- net BCLK: track 106.2 -> 82.6 mm
Other:
- board size 100 x 100 mm -> 193 x 100 mm
