File: draft9.sch (EAGLE design)
At the start: 197 parts, among them Q1 Si2333, Q2 2N7002, Q3 2N7002, Q4 2N7002, Q5 2N7002, Q6 2N7002, Q7 2N7002, SW11 TOUCH_PAD-CIRCLE-15MM, SW2 TOUCH_PAD-CIRCLE-15MM, SW3 TOUCH_PAD-CIRCLE-15MM, SW4 TOUCH_PAD-CIRCLE-15MM, SW5 TOUCH_PAD-CIRCLE-15MM, SW6 TOUCH_PAD-CIRCLE-15MM, SW7 TOUCH_PAD-CIRCLE-15MM, U1 CC85XX, U11 CS4270-TSSOP24, U12 SN74LVC1G80DBV, U2 CC2591, U3 CS2300-MSOP10L, U4 AT32UC3A3-LQFP-144, U6 LTC4088-2, U8 AT42QT1110-TQFP, U9 LM4881, X1 48MHz, X2 12MHz

Commit message: Layout work
Connections:
- net !CS_CC8531: now also U4A.PA07; no longer U4A.PA06
- net !MUTE_L: now also U4X.PX30; no longer U4X.PX31
- net !MUTE_R: now also U4X.PX33; no longer U4X.PX30
- net !RESET_CC8531: now also U4A.PA06; no longer U4A.PA07
- net !RESET_CODEC: now also U4X.PX31; no longer U4X.PX33
Changed lines of the file:
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@@
+</segment>
+<segment>
+<wire x1="431.8" y1="-269.24" x2="426.72" y2="-269.24" width="0.1524" layer="91"/>
+<label x="426.72" y="-269.24" size="1.778" layer="95" rot="R180" xref="yes"/>
+<pinref part="U4" gate="A" pin="PA06"/>
+</segment>
+</net>
+<net name="N$9" class="0">
+<segment>
+<pinref part="C26" gate="G$1" pin="2"/>
+<wire x1="226.06" y1="49.53" x2="229.87" y2="49.53" width="0.1524" layer="91"/>
+<pinref part="SMA" gate="G$1" pin="SIG"/>
+</segment>
+</net>
+<net name="N$28" class="0">
+<segment>
+<pinref part="R5" gate="G$1" pin="1"/>
+<wire x1="-170.18" y1="6.35" x2="-165.1" y2="6.35" width="0.1524" layer="91"/>
+<pinref part="U1" gate="G$1" pin="GIO3"/>
+</segment>
+</net>
+<net name="DIN" class="0">
+<segment>
+<wire x1="-190.5" y1="-24.13" x2="-187.96" y2="-24.13" width="0.1524" layer="91"/>
+<label x="-190.5" y="-24.13" size="1.778" layer="95" rot="R180" xref="yes"/>
+<pinref part="L13" gate="G$1" pin="1"/>
+</segment>
+<segment>
+<pinref part="U11" gate="G$1" pin="DIN"/>
+<wire x1="-180.34" y1="-116.84" x2="-185.42" y2="-116.84" width="0.1524" layer="91"/>
+<label x="-185.42" y="-116.84" size="1.778" layer="95" rot="R180" xref="yes"/>
+</segment>
+<segment>
+<pinref part="U4" gate="X" pin="PX24"/>
+<wire x1="755.65" y1="-377.19" x2="749.3" y2="-377.19" width="0.1524" layer="91"/>
+<label x="749.3" y="-377.19" size="1.778" layer="95" rot="R180" xref="yes"/>
+</segment>
+</net>
+<net name="DOUT" class="0">
+<segment>
+<wire x1="-180.34" y1="-19.05" x2="-190.5" y2="-19.05" width="0.1524" layer="91"/>
+<label x="-190.5" y="-19.05" size="1.778" layer="95" rot="R180" xref="yes"/>
+<pinref part="L11" gate="G$1" pin="1"/>
+</segment>
+<segment>
+<pinref part="U11" gate="G$1" pin="DOUT"/>
+<wire x1="-180.34" y1="-137.16" x2="-185.42" y2="-137.16" width="0.1524" layer="91"/>
+<label x="-185.42" y="-137.16" size="1.778" layer="95" rot="R180" xref="yes"/>
+</segment>
+<segment>
+<pinref part="U4" gate="X" pin="PX25"/>
+<wire x1="755.65" y1="-382.27" x2="749.3" y2="-382.27" width="0.1524" layer="91"/>
+<label x="749.3" y="-382.27" size="1.778" layer="95" rot="R180" xref="yes"/>
+</segment>
+</net>
+<net name="PHONE_R" class="2">
+<segment>
+<pinref part="C39" gate="G$1" pin="2"/>
+<wire x1="-1.27" y1="-204.47" x2="1.27" y2="-204.47" width="0.1524" layer="91"/>
+<label x="1.27" y="-204.47" size="1.778" layer="95" xref="yes"/>
+</segment>
+<segment>
+<wire x1="-130.81" y1="-218.44" x2="-133.35" y2="-218.44" width="0.1524" layer="91"/>
+<label x="-133.35" y="-218.44" size="1.778" layer="95" rot="R180" xref="yes"/>
+<pinref part="PHONE_OUT" gate="G$1" pin="R"/>
+</segment>
+</net>
+<net name="!CS_CC8531" class="0">
+<segment>
+<wire x1="-165.1" y1="39.37" x2="-167.64" y2="39.37" width="0.1524" layer="91"/>
+<label x="-167.64" y="39.37" size="1.778" layer="95" rot="R180" xref="yes"/>
+<pinref part="U1" gate="G$1" pin="!CS"/>
+</segment>
+<segment>
+<pinref part="CC_DEBUG" gate="G$1" pin="5"/>
+<wire x1="-11.43" y1="41.91" x2="-13.97" y2="41.91" width="0.1524" layer="91"/>
+<label x="-13.97" y="41.91" size="1.778" layer="95" rot="R180" xref="yes"/>
 </segment>
 <segment>
@@
 <label x="426.72" y="-274.32" size="1.778" layer="95" rot="R180" xref="yes"/>
 <pinref part="U4" gate="A" pin="PA07"/>
-</segment>
-</net>
-<net name="N$9" class="0">
-<segment>
-<pinref part="C26" gate="G$1" pin="2"/>
-<wire x1="226.06" y1="49.53" x2="229.87" y2="49.53" width="0.1524" layer="91"/>
-<pinref part="SMA" gate="G$1" pin="SIG"/>
-</segment>
-</net>
-<net name="N$28" class="0">
-<segment>
-<pinref part="R5" gate="G$1" pin="1"/>
-<wire x1="-170.18" y1="6.35" x2="-165.1" y2="6.35" width="0.1524" layer="91"/>
-<pinref part="U1" gate="G$1" pin="GIO3"/>
-</segment>
-</net>
-<net name="DIN" class="0">
-<segment>
-<wire x1="-190.5" y1="-24.13" x2="-187.96" y2="-24.13" width="0.1524" layer="91"/>
-<label x="-190.5" y="-24.13" size="1.778" layer="95" rot="R180" xref="yes"/>
-<pinref part="L13" gate="G$1" pin="1"/>
-</segment>
-<segment>
-<pinref part="U11" gate="G$1" pin="DIN"/>
-<wire x1="-180.34" y1="-116.84" x2="-185.42" y2="-116.84" width="0.1524" layer="91"/>
-<label x="-185.42" y="-116.84" size="1.778" layer="95" rot="R180" xref="yes"/>
-</segment>
-<segment>
-<pinref part="U4" gate="X" pin="PX24"/>
-<wire x1="755.65" y1="-377.19" x2="749.3" y2="-377.19" width="0.1524" layer="91"/>
-<label x="749.3" y="-377.19" size="1.778" layer="95" rot="R180" xref="yes"/>
-</segment>
-</net>
-<net name="DOUT" class="0">
-<segment>
-<wire x1="-180.34" y1="-19.05" x2="-190.5" y2="-19.05" width="0.1524" layer="91"/>
-<label x="-190.5" y="-19.05" size="1.778" layer="95" rot="R180" xref="yes"/>
-<pinref part="L11" gate="G$1" pin="1"/>
-</segment>
-<segment>
-<pinref part="U11" gate="G$1" pin="DOUT"/>
-<wire x1="-180.34" y1="-137.16" x2="-185.42" y2="-137.16" width="0.1524" layer="91"/>
-<label x="-185.42" y="-137.16" size="1.778" layer="95" rot="R180" xref="yes"/>
-</segment>
-<segment>
-<pinref part="U4" gate="X" pin="PX25"/>
-<wire x1="755.65" y1="-382.27" x2="749.3" y2="-382.27" width="0.1524" layer="91"/>
-<label x="749.3" y="-382.27" size="1.778" layer="95" rot="R180" xref="yes"/>
-</segment>
-</net>
-<net name="PHONE_R" class="2">
-<segment>
-<pinref part="C39" gate="G$1" pin="2"/>
-<wire x1="-1.27" y1="-204.47" x2="1.27" y2="-204.47" width="0.1524" layer="91"/>
-<label x="1.27" y="-204.47" size="1.778" layer="95" xref="yes"/>
-</segment>
-<segment>
-<wire x1="-130.81" y1="-218.44" x2="-133.35" y2="-218.44" width="0.1524" layer="91"/>
-<label x="-133.35" y="-218.44" size="1.778" layer="95" rot="R180" xref="yes"/>
-<pinref part="PHONE_OUT" gate="G$1" pin="R"/>
-</segment>
-</net>
-<net name="!CS_CC8531" class="0">
-<segment>
-<wire x1="-165.1" y1="39.37" x2="-167.64" y2="39.37" width="0.1524" layer="91"/>
-<label x="-167.64" y="39.37" size="1.778" layer="95" rot="R180" xref="yes"/>
-<pinref part="U1" gate="G$1" pin="!CS"/>
-</segment>
-<segment>
-<pinref part="CC_DEBUG" gate="G$1" pin="5"/>
-<wire x1="-11.43" y1="41.91" x2="-13.97" y2="41.91" width="0.1524" layer="91"/>
-<label x="-13.97" y="41.91" size="1.778" layer="95" rot="R180" xref="yes"/>
-</segment>
-<segment>
-<wire x1="431.8" y1="-269.24" x2="426.72" y2="-269.24" width="0.1524" layer="91"/>
-<label x="426.72" y="-269.24" size="1.778" layer="95" rot="R180" xref="yes"/>
-<pinref part="U4" gate="A" pin="PA06"/>
 </segment>
 </net>
@@
 </segment>
 <segment>
+<pinref part="U4" gate="X" pin="PX31"/>
+<wire x1="900.43" y1="-260.35" x2="905.51" y2="-260.35" width="0.1524" layer="91"/>
+<label x="905.51" y="-260.35" size="1.778" layer="95" xref="yes"/>
+</segment>
+</net>
+<net name="!MUTE_R" class="0">
+<segment>
+<pinref part="U11" gate="G$1" pin="!MUTEB"/>
+<wire x1="-142.24" y1="-121.92" x2="-137.16" y2="-121.92" width="0.1524" layer="91"/>
+<label x="-137.16" y="-121.92" size="1.778" layer="95" xref="yes"/>
+</segment>
+<segment>
 <wire x1="900.43" y1="-270.51" x2="905.51" y2="-270.51" width="0.1524" layer="91"/>
 <label x="905.51" y="-270.51" size="1.778" layer="95" xref="yes"/>
@@
 </segment>
 </net>
-<net name="!MUTE_R" class="0">
-<segment>
-<pinref part="U11" gate="G$1" pin="!MUTEB"/>
-<wire x1="-142.24" y1="-121.92" x2="-137.16" y2="-121.92" width="0.1524" layer="91"/>
-<label x="-137.16" y="-121.92" size="1.778" layer="95" xref="yes"/>
+<net name="!MUTE_L" class="0">
+<segment>
+<pinref part="U11" gate="G$1" pin="!MUTEA"/>
+<wire x1="-142.24" y1="-127" x2="-137.16" y2="-127" width="0.1524" layer="91"/>
+<label x="-137.16" y="-127" size="1.778" layer="95" xref="yes"/>
 </segment>
 <segment>
@@
 </segment>
 </net>
-<net name="!MUTE_L" class="0">
-<segment>
-<pinref part="U11" gate="G$1" pin="!MUTEA"/>
-<wire x1="-142.24" y1="-127" x2="-137.16" y2="-127" width="0.1524" layer="91"/>
-<label x="-137.16" y="-127" size="1.778" layer="95" xref="yes"/>
-</segment>
-<segment>
-<pinref part="U4" gate="X" pin="PX31"/>
-<wire x1="900.43" y1="-260.35" x2="905.51" y2="-260.35" width="0.1524" layer="91"/>
-<label x="905.51" y="-260.35" size="1.778" layer="95" xref="yes"/>
-</segment>
-</net>

Commit message: More layout work
Parts:
- removed R11: 0, 00-EvaLibrary:R-US_R0603
Connections:
- removed net 3.3V: L18.2, L19.2
- removed net AVDD_CODEC1: C14.1, C48.1, L21.1, U4P.VDDANA
- removed net N$50: CC_DEBUG.9, R11.2
- net !CHANGE: now also U4X.PX12; no longer U4X.PX55
- net !CS_TOUCH: now also U4X.PX13; no longer U4X.PX21
- net AVDD_CODEC: now also C14.1, C48.1, L21.1, U4P.VDDANA
- net D3.3V: now also L18.2, L19.2; no longer R11.1
Changed lines of the file:
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@@
 <part name="C65" library="rcl" deviceset="C-EU" device="C0603" value="2.2u"/>
 <part name="L18" library="SparkFun-Passives" deviceset="INDUCTOR" device="0603" value="BEAD"/>
-<part name="P+3" library="SparkFun" deviceset="3.3V" device=""/>
 <part name="U9" library="00-EvaLibrary" deviceset="LM4881" device=""/>
 <part name="C33" library="rcl" deviceset="C-EU" device="C0603" value="1u"/>
@@
 <part name="C57" library="rcl" deviceset="C-EU" device="C0603" value="2.2u"/>
 <part name="L19" library="SparkFun-Passives" deviceset="INDUCTOR" device="0603" value="BEAD"/>
-<part name="P+9" library="SparkFun" deviceset="3.3V" device=""/>
 <part name="R44" library="rcl" deviceset="R-US_" device="R0603" value="100"/>
 <part name="JTAG" library="00-EvaLibrary" deviceset="HEADER-10P" device="-SMD-MALE2"/>
@@
 <part name="D3.3V3" library="00-EvaLibrary" deviceset="D3.3V" device=""/>
 <part name="D3.3V4" library="00-EvaLibrary" deviceset="D3.3V" device=""/>
-<part name="D3.3V5" library="00-EvaLibrary" deviceset="D3.3V" device=""/>
 <part name="DGND4" library="00-EvaLibrary" deviceset="DGND" device=""/>
 <part name="DGND5" library="00-EvaLibrary" deviceset="DGND" device=""/>
@@
 <part name="C102" library="rcl" deviceset="C-EU" device="C0603" value="100n"/>
 <part name="DGND82" library="00-EvaLibrary" deviceset="DGND" device=""/>
-<part name="R11" library="00-EvaLibrary" deviceset="R-US_" device="R0603" value="0"/>
 <part name="SW2" library="00-EvaLibrary" deviceset="TOUCH_PAD" device="-CIRCLE-15MM" value="TOUCH_PAD-CIRCLE-15MM"/>
 <part name="SW3" library="00-EvaLibrary" deviceset="TOUCH_PAD" device="-CIRCLE-15MM" value="TOUCH_PAD-CIRCLE-15MM"/>
@@
 <part name="R26" library="00-EvaLibrary" deviceset="R-US_" device="R0603" value="0"/>
 <part name="AGND18" library="00-EvaLibrary" deviceset="AGND" device=""/>
+<part name="D3.3V5" library="00-EvaLibrary" deviceset="D3.3V" device=""/>
+<part name="D3.3V9" library="00-EvaLibrary" deviceset="D3.3V" device=""/>
 </parts>
 <sheets>
@@
 <attribute name="VALUE" x="384.81" y="-185.42" size="1.778" layer="96"/>
 </instance>
-<instance part="P+3" gate="G$1" x="383.54" y="-175.26" smashed="yes">
-<attribute name="VALUE" x="382.524" y="-171.704" size="1.778" layer="96"/>
-</instance>
 <instance part="U9" gate="G$1" x="-35.56" y="-186.69"/>
 <instance part="C33" gate="G$1" x="-50.8" y="-196.85" smashed="yes">
@@
 <attribute name="VALUE" x="335.28" y="-177.8" size="1.778" layer="96"/>
 </instance>
-<instance part="P+9" gate="G$1" x="334.01" y="-167.64" smashed="yes">
-<attribute name="VALUE" x="332.994" y="-164.084" size="1.778" layer="96"/>
-</instance>
 <instance part="R44" gate="G$1" x="613.41" y="-167.64" smashed="yes" rot="R90">
 <attribute name="NAME" x="614.68" y="-166.37" size="1.778" layer="95"/>
@@
 <instance part="D3.3V3" gate="G$1" x="-53.34" y="99.06"/>
 <instance part="D3.3V4" gate="G$1" x="1.27" y="54.61"/>
-<instance part="D3.3V5" gate="G$1" x="-45.72" y="31.75"/>
 <instance part="DGND4" gate="G$1" x="-195.58" y="99.06"/>
 <instance part="DGND5" gate="G$1" x="-189.23" y="90.17"/>
@@
 </instance>
 <instance part="DGND82" gate="G$1" x="1012.19" y="-271.78"/>
-<instance part="R11" gate="G$1" x="-31.75" y="31.75" smashed="yes">
-<attribute name="NAME" x="-34.29" y="33.2486" size="1.778" layer="95"/>
-<attribute name="VALUE" x="-34.29" y="28.448" size="1.778" layer="96"/>
-</instance>
 <instance part="SW2" gate="G$1" x="412.75" y="8.89"/>
 <instance part="SW3" gate="G$1" x="412.75" y="-5.08"/>
@@
 </instance>
 <instance part="AGND18" gate="G$1" x="-35.56" y="-219.71"/>
+<instance part="D3.3V5" gate="G$1" x="334.01" y="-167.64"/>
+<instance part="D3.3V9" gate="G$1" x="383.54" y="-175.26"/>
 </instances>
 <busses>
 </busses>
 <nets>
-<net name="3.3V" class="1">
-<segment>
-<pinref part="L18" gate="G$1" pin="2"/>
-<pinref part="P+3" gate="G$1" pin="3.3V"/>
-</segment>
-<segment>
-<pinref part="L19" gate="G$1" pin="2"/>
-<pinref part="P+9" gate="G$1" pin="3.3V"/>
-</segment>
-</net>
 <net name="PA_EN" class="0">
 <segment>
@@
 </segment>
 </net>
-<net name="N$50" class="0">
-<segment>
-<pinref part="CC_DEBUG" gate="G$1" pin="9"/>
-<wire x1="-26.67" y1="31.75" x2="-11.43" y2="31.75" width="0.1524" layer="91"/>
-<pinref part="R11" gate="G$1" pin="2"/>
-</segment>
-</net>
 <net name="VBUS" class="1">
 <segment>
@@
 <junction x="-35.56" y="-157.48"/>
 </segment>
+<segment>
+<pinref part="C14" gate="G$1" pin="1"/>
+<pinref part="L21" gate="G$1" pin="1"/>
+<junction x="734.06" y="-196.85"/>
+<wire x1="734.06" y1="-196.85" x2="725.17" y2="-196.85" width="0.1524" layer="91"/>
+<pinref part="U4" gate="P" pin="VDDANA"/>
+<wire x1="725.17" y1="-196.85" x2="713.74" y2="-196.85" width="0.1524" layer="91"/>
+<wire x1="713.74" y1="-212.09" x2="713.74" y2="-196.85" width="0.1524" layer="91"/>
+<pinref part="C48" gate="G$1" pin="1"/>
+<junction x="725.17" y="-196.85"/>
+<label x="713.74" y="-195.58" size="1.778" layer="95"/>
+</segment>
 </net>
 <net name="DVDD_CODEC" class="0">
@@
 </segment>
 <segment>
-<wire x1="900.43" y1="-382.27" x2="905.51" y2="-382.27" width="0.1524" layer="91"/>
-<label x="905.51" y="-382.27" size="1.778" layer="95" xref="yes"/>
-<pinref part="U4" gate="X" pin="PX55"/>
+<wire x1="755.65" y1="-316.23" x2="750.57" y2="-316.23" width="0.1524" layer="91"/>
+<label x="750.57" y="-316.23" size="1.778" layer="95" rot="R180" xref="yes"/>
+<pinref part="U4" gate="X" pin="PX12"/>
 </segment>
 </net>
@@
 </segment>
 <segment>
-<wire x1="755.65" y1="-361.95" x2="748.03" y2="-361.95" width="0.1524" layer="91"/>
-<label x="748.03" y="-361.95" size="1.778" layer="95" rot="R180" xref="yes"/>
-<pinref part="U4" gate="X" pin="PX21"/>
+<wire x1="755.65" y1="-321.31" x2="748.03" y2="-321.31" width="0.1524" layer="91"/>
+<label x="748.03" y="-321.31" size="1.778" layer="95" rot="R180" xref="yes"/>
+<pinref part="U4" gate="X" pin="PX13"/>
 </segment>
 </net>
@@
 </segment>
 <segment>
-<wire x1="-45.72" y1="31.75" x2="-36.83" y2="31.75" width="0.1524" layer="91"/>
-<pinref part="D3.3V5" gate="G$1" pin="D3.3V"/>
-<pinref part="R11" gate="G$1" pin="1"/>
-</segment>
-<segment>
 <pinref part="L3" gate="G$1" pin="2"/>
 <pinref part="D3.3V6" gate="G$1" pin="D3.3V"/>
@@
 <pinref part="D3.3V8" gate="G$1" pin="D3.3V"/>
 </segment>
+<segment>
+<pinref part="L19" gate="G$1" pin="2"/>
+<pinref part="D3.3V5" gate="G$1" pin="D3.3V"/>
+</segment>
+<segment>
+<pinref part="L18" gate="G$1" pin="2"/>
+<pinref part="D3.3V9" gate="G$1" pin="D3.3V"/>
+</segment>
 </net>
 <net name="N$88" class="0">
@@
 </segment>
 </net>
-<net name="AVDD_CODEC1" class="0">
-<segment>
-<pinref part="C14" gate="G$1" pin="1"/>
-<pinref part="L21" gate="G$1" pin="1"/>
-<junction x="734.06" y="-196.85"/>
-<wire x1="734.06" y1="-196.85" x2="725.17" y2="-196.85" width="0.1524" layer="91"/>
-<pinref part="U4" gate="P" pin="VDDANA"/>
-<wire x1="725.17" y1="-196.85" x2="713.74" y2="-196.85" width="0.1524" layer="91"/>
-<wire x1="713.74" y1="-212.09" x2="713.74" y2="-196.85" width="0.1524" layer="91"/>
-<pinref part="C48" gate="G$1" pin="1"/>
-<junction x="725.17" y="-196.85"/>
-</segment>
-</net>

Commit message: Did a whole lot of things
Parts:
- removed C100, C101, C102: 100n, rcl:C-EUC0603
- removed C96: 1n, rcl:C-EUC0603
- removed C97: 1u, rcl:C-EUC0603
- removed L18: BEAD, SparkFun-Passives:INDUCTOR0603
- removed MICROSD: MICROSD104031-0811, 00-EvaLibrary:MICROSD104031-0811
- removed Q1: Si2333, SparkFun-DiscreteSemi:MOSFET-PCHANNELSMD
- removed R23: 100K, rcl:R-US_R0603
- removed R44: 100, rcl:R-US_R0603
- removed SW11, SW2, SW3, SW4, SW5, SW6, SW7: TOUCH_PAD-CIRCLE-15MM, 00-EvaLibrary:TOUCH_PAD-CIRCLE-15MM
- removed U12: SN74LVC1G80DBV, 00-EvaLibrary:SN74LVC1G80DBV
- added AVR1: (no value), SparkFun-LED:LED1206
- added BUTTON, NEXT, PLAY/PAUSE, PREV, STOP, VOL+, VOL-, WIRELESS: TOUCH_PAD-CIRCLE-10MM, 00-EvaLibrary:TOUCH_PAD-CIRCLE-10MM
- added C44, C46: 100n, 00-EvaLibrary:C-EUC0603
- added C47: 10u, 00-EvaLibrary:C-EUC0603
- added C55, C67, C68: 1u, 00-EvaLibrary:C-EUC0603
- added C56, C69: 1n, 00-EvaLibrary:C-EUC0603
- added C62: 2.2u, 00-EvaLibrary:C-EUC0603
- added C66: 220u, 00-EvaLibrary:C-EUC1210
- added GPIO: TACT_SWITCH-PTS-525, 00-EvaLibrary:TACT_SWITCH-PTS-525
- added L16: BEAD, SparkFun-Passives:INDUCTOR0603
- added R11: 332, 00-EvaLibrary:R-US_R0603
- added R30, R32: 4.64K, 00-EvaLibrary:R-US_R0603
- added R38: 681, 00-EvaLibrary:R-US_R0603
- added R39: 4.53K, 00-EvaLibrary:R-US_R0603
- added R40, R41: 1K, 00-EvaLibrary:R-US_R0603
- added SD1: MICROSD104031-0811, 00-EvaLibrary:MICROSD104031-0811
- added SERIAL: HEADER-6X1-961106-5500, 00-EvaLibrary:HEADER-6X1-961106-5500
- added U7: TLV700DDC, 00-EvaLibrary:TLV700DDC
- C1, C2: value 2.2u -> 100n; device rcl:C-EUC0603 -> 00-EvaLibrary:C-EUC0603
- C10: value 220p -> 1n; device rcl:C-EUC0603 -> 00-EvaLibrary:C-EUC0603
- C11, C15, C19, C31, C32, C40, C41, C42, C6, C64, C79: device rcl:C-EUC0603 -> 00-EvaLibrary:C-EUC0603
- C12, C7: value 100n -> 1n; device rcl:C-EUC0603 -> 00-EvaLibrary:C-EUC0603
- C13: value 2.2u -> 10p; device rcl:C-EUC0603 -> 00-EvaLibrary:C-EUC0603
- C14, C85, C95: value 1u -> 100n; device rcl:C-EUC0603 -> 00-EvaLibrary:C-EUC0603
- C16: value 10p -> 2.2u; device rcl:C-EUC0603 -> 00-EvaLibrary:C-EUC0603
- C17, C20, C86: value 1n -> 100n; device rcl:C-EUC0603 -> 00-EvaLibrary:C-EUC0603
- C18: value 10p -> 1u; device rcl:C-EUC0603 -> 00-EvaLibrary:C-EUC0603
- C21: value 18p -> 6.8p_HF; device rcl:C-EUC0603 -> 00-EvaLibrary:C-EUC0603
- C22: value 1n -> 100p_HF; device rcl:C-EUC0603 -> 00-EvaLibrary:C-EUC0603
- C23: value 1u -> 1.2p_HF; device rcl:C-EUC0603 -> 00-EvaLibrary:C-EUC0603
- C24: value 15p -> 1.8p_HF; device rcl:C-EUC0603 -> 00-EvaLibrary:C-EUC0603
- C25: value 6.8p_HF -> 1u; device rcl:C-EUC0603 -> 00-EvaLibrary:C-EUC0603
- C26: value 100p_HF -> 27p; device rcl:C-EUC0603 -> 00-EvaLibrary:C-EUC0603
- C27: value 1.2p_HF -> 27p; device rcl:C-EUC0603 -> 00-EvaLibrary:C-EUC0603
- C28: value 1.8p_HF -> 1u; device rcl:C-EUC0603 -> 00-EvaLibrary:C-EUC0603
- C29: value 15p -> 100n; device rcl:C-EUC0603 -> 00-EvaLibrary:C-EUC0603
- C3: value 1u -> 2.2u; device rcl:C-EUC0603 -> 00-EvaLibrary:C-EUC0603
- C30: value 10n -> 100n; device rcl:C-EUC0603 -> 00-EvaLibrary:C-EUC0603
- C33, C49: value 1u -> 1n; device rcl:C-EUC0603 -> 00-EvaLibrary:C-EUC0603
- C34, C48, C63, C77: value 100n -> 1u; device rcl:C-EUC0603 -> 00-EvaLibrary:C-EUC0603
- C35, C43, C58: value 10n -> 1n; device rcl:C-EUC0603 -> 00-EvaLibrary:C-EUC0603
- C36: value 220u -> 470n; device 00-EvaLibrary:C-EUC1210 -> 00-EvaLibrary:C-EUC0603
- C37, C54: value 100n -> 2.2u
- C38: value 100n -> 470n; device rcl:C-EUC0603 -> 00-EvaLibrary:C-EUC0603
- C39: value 220u -> 100n; device 00-EvaLibrary:C-EUC1210 -> 00-EvaLibrary:C-EUC0603
- C4: value 100n -> 100n_HF; device rcl:C-EUC0603 -> 00-EvaLibrary:C-EUC0603
- C45: value 1n -> 10u; device rcl:C-EUC0603 -> 00-EvaLibrary:C-EUC0603
- C5: value 100n -> 220p_HF; device rcl:C-EUC0603 -> 00-EvaLibrary:C-EUC0603
- C50: value 1n -> 1u; device rcl:C-EUC0603 -> 00-EvaLibrary:C-EUC0603
- C51: value 10u -> 1n
- C52, C80: value 10u -> 1u; device rcl:C-EUC0603 -> 00-EvaLibrary:C-EUC0603
- C53: value 10u -> 220u; device rcl:C-EUC0603 -> 00-EvaLibrary:C-EUC1210
- C57, C65: value 2.2u -> 1u; device rcl:C-EUC0603 -> 00-EvaLibrary:C-EUC0603
- C59, C60, C61: value 10n -> 10u; device rcl:C-EUC0603 -> 00-EvaLibrary:C-EUC0603
- C70: value 470n -> 10u
- C71: value 470n -> 1u; device rcl:C-EUC0603 -> 00-EvaLibrary:C-EUC0603
- C72: value 10p -> 1u
- C73: value 10p -> 100n
- C74: value 100n -> 1u
- C75: value 10p -> 1n
- C76: value 10u -> 10p; device rcl:C-EUC0603 -> 00-EvaLibrary:C-EUC0603
- C78: value 10u -> 1n; device rcl:C-EUC0603 -> 00-EvaLibrary:C-EUC0603
- C8: value 100n -> 10p; device rcl:C-EUC0603 -> 00-EvaLibrary:C-EUC0603
- C81, C82: value 470n -> 100n; device rcl:C-EUC0603 -> 00-EvaLibrary:C-EUC0603
- C83: value 1u -> 10p; device rcl:C-EUC0603 -> 00-EvaLibrary:C-EUC0603
- C84: value 1n -> 10p; device rcl:C-EUC0603 -> 00-EvaLibrary:C-EUC0603
- C87, C89, C91, C93: value 1u -> 10n; device rcl:C-EUC0603 -> 00-EvaLibrary:C-EUC0603
- C88, C90, C92, C94: value 1n -> 10n; device rcl:C-EUC0603 -> 00-EvaLibrary:C-EUC0603
- C9: value 100n -> 18p; device rcl:C-EUC0603 -> 00-EvaLibrary:C-EUC0603
- C98: value 1n -> 470n; device rcl:C-EUC0603 -> 00-EvaLibrary:C-EUC0603
- C99: value 1u -> 470n; device rcl:C-EUC0603 -> 00-EvaLibrary:C-EUC0603
- L1, L2: value BEAD -> BEAD_HF; device SparkFun-Passives:INDUCTOR0603 -> 00-EvaLibrary:INDUCTOR0603
- L10: value 1.5n_HF -> 6.8n; device SparkFun-Passives:INDUCTOR0603 -> 00-EvaLibrary:INDUCTOR0603
- L11, L13, L14, L19, L20, L21, L3, L9: device SparkFun-Passives:INDUCTOR0603 -> 00-EvaLibrary:INDUCTOR0603
- L17: value 3.3u -> BEAD; device 00-EvaLibrary:IFSC-1111AB-01 -> 00-EvaLibrary:INDUCTOR0603
- L4: value 6.8n -> 2.2n_HF; device SparkFun-Passives:INDUCTOR0603 -> 00-EvaLibrary:INDUCTOR0603
- L5: value 6.8n -> 3.9n_HF; device SparkFun-Passives:INDUCTOR0603 -> 00-EvaLibrary:INDUCTOR0603
- L6: value 6.8n -> 1.5n_HF; device SparkFun-Passives:INDUCTOR0603 -> 00-EvaLibrary:INDUCTOR0603
- L7: value 2.2n_HF -> 6.8n; device SparkFun-Passives:INDUCTOR0603 -> 00-EvaLibrary:INDUCTOR0603
- L8: value 3.9n_HF -> 6.8n; device SparkFun-Passives:INDUCTOR0603 -> 00-EvaLibrary:INDUCTOR0603
- R1, R2: value 0 -> 4.32K
- R12: value 20K -> 100
- R13, R16: value 20K -> 1M
- R14: value 4.7K -> 20K; device rcl:R-US_R0603 -> 00-EvaLibrary:R-US_R0603
- R15: value 20K -> 39
- R17, R25, R5: device rcl:R-US_R0603 -> 00-EvaLibrary:R-US_R0603
- R18: value 330 -> 10K
- R19: value 8.2 -> 100K
- R20: value 2.94K -> 100K
- R21: value 1K -> 20K
- R22: value 1M -> 100K; device rcl:R-US_R0603 -> 00-EvaLibrary:R-US_R0603
- R24: value 1M -> 0; device rcl:R-US_R0603 -> 00-EvaLibrary:R-US_R0603
- R27: value 6.8K -> 6.81K; device rcl:R-US_R0603 -> 00-EvaLibrary:R-US_R0603
- R28: value 4.7K -> 100K; device rcl:R-US_R0603 -> 00-EvaLibrary:R-US_R0603
- R29, R33, R34, R35: value 4.7K -> 4.64K; device rcl:R-US_R0603 -> 00-EvaLibrary:R-US_R0603
- R3: value 100 -> 56.2K; device rcl:R-US_R0603 -> 00-EvaLibrary:R-US_R0603
- R31: value 10K -> 4.64K; device rcl:R-US_R0603 -> 00-EvaLibrary:R-US_R0603
- R36: value 100K -> 4.64K; device rcl:R-US_R0603 -> 00-EvaLibrary:R-US_R0603
- R37: value 4.7K -> 10K; device rcl:R-US_R0603 -> 00-EvaLibrary:R-US_R0603
- R4: value 56k -> 100; device rcl:R-US_R0603 -> 00-EvaLibrary:R-US_R0603
- R6: value 39 -> 10K; device rcl:R-US_R0603 -> 00-EvaLibrary:R-US_R0603
- R7: value 10K -> 20K; device rcl:R-US_R0603 -> 00-EvaLibrary:R-US_R0603
- R8: value 4.3K -> 100; device rcl:R-US_R0603 -> 00-EvaLibrary:R-US_R0603
- R9: value 4.3K -> 20K; device rcl:R-US_R0603 -> 00-EvaLibrary:R-US_R0603
- U1: value CC85XX -> CC2591; device 00-EvaLibrary:CC85XX -> 00-EvaLibrary:CC2591
- U10: value (none) -> AT32UC3A3-LQFP-144; device 00-EvaLibrary:MCP1826-SOT223 -> 00-EvaLibrary:AT32UC3A3-LQFP-144
- U11: value CS4270-TSSOP24 -> AT42QT1110-QFN-32; device 00-EvaLibrary:CS4270-TSSOP24 -> 00-EvaLibrary:AT42QT1110-QFN-32
- U2: value CC2591 -> CC85XX; device 00-EvaLibrary:CC2591 -> 00-EvaLibrary:CC85XX
- U3: value CS2300-MSOP10L -> CS4270-TSSOP24; device 00-EvaLibrary:CS2300-MSOP10L -> 00-EvaLibrary:CS4270-TSSOP24
- U4: value AT32UC3A3-LQFP-144 -> LM4881; device 00-EvaLibrary:AT32UC3A3-LQFP-144 -> 00-EvaLibrary:LM4881
- U6: value LTC4088-2 -> BQ2409XDGQ; device 00-EvaLibrary:LTC4088-1/2 -> 00-EvaLibrary:BQ2409XDGQ
- U8: value AT42QT1110-TQFP -> SN74LVC1G80DBV; device 00-EvaLibrary:AT42QT1110-TQFP -> 00-EvaLibrary:SN74LVC1G80DBV
- U9: value LM4881 -> CS2300-MSOP10L; device 00-EvaLibrary:LM4881 -> 00-EvaLibrary:CS2300-MSOP10L
- renumbered CC8531 to CC1, RESET1 to RESET, USB2 to USB
Connections:
- removed net !AVR_LED: AVR.C, U4X.PX08
- removed net !CS_SD: MICROSD.!CS, U4B.PB09
- removed net N$36: L17.1, U6.SW
- removed net N$37: R21.2, U6.C/X, U6.PROG
- removed net N$38: R19.2, R20.2, U6.CLRPROG
- removed net N$48: C54.1, R19.1
- new net !AVR_LED0: AVR.C, U10X.PX08
- new net !AVR_LED1: AVR1.C, U10X.PX15
- new net !GPIO: GPIO.2, U10X.PX46
- new net AUX_VDD2: LED_LL.A, LED_LR.A, LED_UL.A, LED_UR.A, TO_MAIN2.1, TO_MAIN2.2
- new net AUX_VSS1: Q2.S, Q3.S, Q4.S, Q5.S, Q6.S, Q7.S, TO_MAIN2.10, TO_MAIN2.9
- new net MCI-CLK: SD1.CLK/SCLK, U10A.PA27
- new net MCI-CMD: R22.1, SD1.CMD/MOSI, U10A.PA28
- new net MCI-DATA0: R20.1, SD1.DAT0/MISO, U10A.PA29
- new net MCI-DATA1: SD1.DAT1/NC, U10A.PA30
- new net MCI-DATA2: SD1.DAT2/NC, U10A.PA31
- new net MCI-DATA3: SD1.CD/DAT3/!CS, U10B.PB00
- new net N$11: PLAY/PAUSE.P$1, R36.2
- new net N$17: C94.1, U11.SNS7/DETECT1
- new net N$44: R38.2, U6.ISET
- new net N$50: F1.2, L21.2, U5.VIN
- new net N$6: C94.2, R36.1, U11.SNS7K/DETECT0
- new net N$66: R37.2, U6.TS
- new net N$69: R39.2, U6.PRETERM
- net !CHANGE: now also TO_AUX2.9, U10X.PX12; no longer TO_AUX1.9, U4X.PX12
- net !CS_CC8531: now also U10A.PA07, U2.!CS; no longer U1.!CS, U4A.PA07
- net !CS_CLOCK: now also U10A.PA14, U9.AD0/!CS; no longer U3.AD0/!CS, U4X.PX54
- net !CS_CODEC: now also U10X.PX32, U3.AD0/!CS; no longer U11.AD0/!CS, U4X.PX29
- net !CS_TOUCH: now also TO_AUX2.7, U10X.PX38; no longer TO_AUX1.7, U4X.PX13
- net !MUTE_L: now also U10X.PX30, U3.!MUTEA; no longer U11.!MUTEA, U4X.PX30
- net !MUTE_R: now also U10X.PX33, U3.!MUTEB; no longer U11.!MUTEB, U4X.PX33
- net !PAIR: now also U10A.PA13, U2.GIO1; no longer U1.GIO1, U4A.PA13
- net !RESET: now also C73.1, R18.1, U10M.!RESET; no longer C74.1, R7.1, U4M.!RESET
- net !RESET_CC8531: now also L7.2, U10A.PA06; no longer L4.2, U4A.PA06
- net !RESET_CODEC: now also U10X.PX31, U3.!RESET; no longer U11.!RESET, U4X.PX31
- net !SD_CARD: now also SD1.SWB, U10B.PB01; no longer MICROSD.SWA, U4A.PA30
- net A3.3V: now also C70.1, L15.2, L20.2, U7.VOUT; no longer C76.1, L14.2, L21.2, U10.VOUT
- net AGND: now also C30.2, C39.2, C44.2, C45.2, C46.2, C47.2, C63.2, C64.2, C65.2, C70.2, C71.2, C98.2, C99.2, R19.1, R24.2, U10P.GNDANA, U3.AGND, U4.VSS, U7.GND; no longer C14.2, C33.2, C34.2, C38.2, C48.2, C76.2, C77.2, C78.2, C79.2, C80.2, R1.2, R23.1, U10.GND, U11.AGND, U4P.GNDANA, U9.VSS
- net ALL_GND: now also C59.2, C60.2, R24.1, R26.1, R37.1, R38.1, R39.1, U6.ISET2, U6.VSS; no longer C51.2, C52.2, C54.2, R1.1, R2.1, R20.1, R21.1, U6.D1, U6.D2, U6.GND, U6.NTC
- net AUDIO: now also C53.1, R7.1, U10A.PA17, U4.OUTA; no longer C36.1, R12.1, U4A.PA17, U9.OUTA
- net AUX_!CHANGE: now also U11.!CHANGE; no longer U8.!CHANGE
- net AUX_BLUE_TOP: now also Q6.G; no longer Q4.G
- net AUX_CS: now also U11.!SS; no longer U8.!SS
- net AUX_GREEN_BOT: now also Q5.G; no longer Q6.G
- net AUX_GREEN_TOP: now also Q4.G; no longer Q3.G
- net AUX_MISO: now also U11.MISO; no longer U8.MISO
- net AUX_MOSI: now also U11.MOSI; no longer U8.MOSI
- net AUX_RED_BOT: now also Q3.G; no longer Q5.G
- net AUX_SCLK: now also U11.SCK; no longer U8.SCK
- net AUX_VDD: now also C85.1, C86.1, R28.2, U11.VDD; no longer C63.1, C64.1, LED_LL.A, LED_LR.A, LED_UL.A, LED_UR.A, R36.2, TO_MAIN2.1, TO_MAIN2.2, U8.VDD
- net AUX_VSS: now also C85.2, C86.2, U11.VSS; no longer C63.2, C64.2, Q2.S, Q3.S, Q4.S, Q5.S, Q6.S, Q7.S, TO_MAIN2.10, TO_MAIN2.9, U8.VSS
- net AVDD: now also C1.1, C13.1, C14.1, C3.1, C4.1, C5.1, C7.1, L1.1, R1.2, U1.AVDD_BIAS, U1.AVDD_LNA, U1.AVDD_PA1, U1.AVDD_PA2, U2.AVDD1, U2.AVDD2, U2.AVDD3, U2.AVDD4, U2.AVDD5, U2.AVDD6; no longer C11.1, C16.1, C17.1, C18.1, C2.1, C21.1, C22.1, L3.1, R9.2, U1.AVDD1, U1.AVDD2, U1.AVDD3, U1.AVDD4, U1.AVDD5, U1.AVDD6, U2.AVDD_BIAS, U2.AVDD_LNA, U2.AVDD_PA1, U2.AVDD_PA2
- net AVDD_CODEC: now also C30.1, C39.1, C64.1, C65.1, L15.1, L20.1, R10.2, R13.2, R16.2, U10P.VDDANA, U3.VA, U4.VDD; no longer C14.1, C34.1, C38.1, C48.1, L14.1, L21.1, R22.2, R24.2, R31.2, U11.VA, U4P.VDDANA, U9.VDD
- net AVR_VDD: now also C32.1, C33.1, C34.1, C35.1, C37.1, C42.1, C43.1, C48.1, C51.1, C55.1, C56.1, C57.1, C58.1, C72.1, C74.1, C75.1, C77.1, C78.1, L16.1, R18.2, R20.2, R22.2, R5.2, R8.2, SD1.VDD, U10P.VDDIN, U10P.VDDIO; no longer C100.1, C102.1, C13.1, C83.1, C84.1, C85.1, C86.1, C87.1, C88.1, C89.1, C90.1, C91.1, C92.1, C93.1, C94.1, C96.1, C97.1, C98.1, C99.1, L20.1, MICROSD.VDD, R44.2, R7.2, U12.VCC, U3.VD, U4P.VDDIN, U4P.VDDIO
- net BAT: now also C60.1, F1.1, R11.2, U2.VBAT, U6.OUT; no longer Q1.S, U1.VBAT, U6.BAT
- net BCLK: now also L9.1, U10X.PX23, U10X.PX28, U10X.PX34, U10X.PX35, U3.BCLK; no longer L6.1, U11.BCLK, U4X.PX23, U4X.PX28, U4X.PX34, U4X.PX35
- net BLUE_BOT: now also TO_AUX1.8, U10X.PX18; no longer TO_AUX2.8, U4X.PX18
- net BLUE_TOP: now also TO_AUX1.3, U10X.PX14; no longer TO_AUX2.3, U4X.PX14
- net CTS: now also SERIAL.5, U10X.PX02; no longer U4X.PX02
- net D+_UC: now also R15.2, U10M.D+_HS; no longer R17.2, U4M.D+_HS
- net D-_UC: now also R17.2, U10M.D-_HS; no longer R6.2, U4M.D-_HS
- net D3.3V: now also C61.1, C79.1, C80.1, C81.1, L14.2, L16.2, L17.2, R12.2, U8.VCC, U9.VD; no longer C53.1, L15.2, L18.2, L20.2, R3.2
- net DAC0_N: now also U10A.PA04; no longer U4A.PA04
- net DAC0_P: now also U10A.PA03; no longer U4A.PA03
- net DAC1_N: now also U10A.PA24; no longer U4A.PA24
- net DAC1_P: now also U10A.PA23; no longer U4A.PA23
- net DGND: now also C14.2, C25.2, C26.2, C33.2, C34.2, C35.2, C43.2, C48.2, C51.2, C54.2, C55.2, C56.2, C58.2, C61.2, C62.2, C68.2, C69.2, C76.2, C77.2, C78.2, C79.2, C80.2, C81.2, C82.2, GPIO.4, L6.1, R2.1, R26.2, R3.1, R6.1, SD1.GND, SD1.SWA, SERIAL.6, TO_AUX1.9, TO_AUX2.6, TO_AUX2.8, U10P.GNDCORE, U10P.GNDIO, U10P.GNDPLL, U2.AD2/GIO9, U2.GIO12, U2.GIO13, U2.SCL/GIO10, U2.SDA/GIO11, U3.DGND, U8.GND, U9.FILTN, U9.GND; no longer C100.2, C101.2, C102.2, C21.2, C22.2, C45.2, C53.2, C65.2, C85.2, C86.2, C87.2, C88.2, C89.2, C90.2, C91.2, C92.2, C93.2, C94.2, C96.2, C97.2, C98.2, C99.2, L10.1, MICROSD.GND, MICROSD.SWB, R10.1, R2.2, R4.1, R8.1, TO_AUX1.6, TO_AUX1.8, TO_AUX2.9, U11.DGND, U12.GND, U3.FILTN, U3.GND, U4P.GNDCORE, U4P.GNDIO, U4P.GNDPLL
- net DIN: now also U10X.PX24, U3.DIN; no longer U11.DIN, U4X.PX24
- net DOUT: now also U10X.PX25, U3.DOUT; no longer U11.DOUT, U4X.PX25
- net DVDD_CODEC: now also C28.1, C29.1, L14.1, U3.VD, U3.VLC; no longer C32.1, C37.1, L15.1, U11.VD, U11.VLC
- net GREEN_BOT: now also TO_AUX1.6, U10A.PA09; no longer TO_AUX2.6, U4A.PA09
- net GREEN_TOP: now also TO_AUX1.5, U10X.PX50; no longer TO_AUX2.5, U4X.PX50
- net IN_L: now also C38.1, R19.2; no longer C82.1, R23.2
- net IN_R: now also C36.1; no longer C81.1
- net IOVDD: now also C11.1, C16.1, C17.1, C18.1, C2.1, L3.1, U2.DVDD, U2.IOVDD1, U2.IOVDD2, U2.IOVDD3, U2.IOVDD4; no longer C1.1, C3.1, C4.1, C5.1, C7.1, L1.1, U1.DVDD, U1.IOVDD1, U1.IOVDD2, U1.IOVDD3, U1.IOVDD4
- net LINEIN_SENSE: now also R13.1, U10A.PA19; no longer R22.1, U4A.PA19
- net LNA_EN: now also U1.EN, U2.XLNAEN; no longer U1.XLNAEN, U2.EN
- net MCLK: now also L8.1, U3.MCLK, U8.CLK, U9.CLK_OUT; no longer R26.1, U11.MCLK, U12.CLK, U3.CLK_OUT
- net MISO0: now also U10A.PA11, U2.MISO, U3.SDA/MISO; no longer TO_AUX1.3, U1.MISO, U11.SDA/MISO, U4A.PA11
- net MISO1: now also TO_AUX2.3, U10B.PB08; no longer MICROSD.MISO, U4B.PB08
- net MOSI0: now also U10A.PA10, U2.MOSI, U3.AD1/MOSI, U9.SDA/MOSI; no longer TO_AUX1.5, U1.MOSI, U11.AD1/MOSI, U4A.PA10
- net MOSI1: now also TO_AUX2.5, U10B.PB10; no longer MICROSD.MOSI, U3.SDA/MOSI, U4B.PB10
- net N$1: now also C26.1, U2.X1; no longer C29.1, U1.X1
- net N$10: now also AVR1.A, R5.1; no longer L5.1, R26.2
- net N$12: now also R8.1; no longer R44.1
- net N$13: now also L4.1, U1.ANT; no longer L7.1, U2.ANT
- net N$14: now also C23.1, L4.2, L5.1; no longer C27.1, L7.2, L8.1
- net N$15: now also C21.1, L5.2; no longer C25.1, L8.2
- net N$16: now also C21.2, C22.1, C24.1, L6.2; no longer C25.2, C26.1, C28.1, L10.2
- net N$18: now also U2.XPAEN; no longer U1.XPAEN
- net N$19: now also R3.2, U2.RBIAS; no longer R4.2, U1.RBIAS
- net N$2: now also C27.1, U2.X0; no longer C24.1, U1.X0
- net N$20: now also C52.2, C98.1, R9.2; no longer C70.2, R13.2
- net N$21: now also C25.1, U2.DCPL; no longer C23.1, U1.DCPL
- net N$22: now also C71.1, L21.1, U7.EN, U7.VIN; no longer F1.2, U10.VIN, U5.VIN
- net N$23: now also L8.2, U2.MCLK/GIO4; no longer L5.2, U1.MCLK/GIO4
- net N$24: now also C67.2, C99.1, R14.2; no longer C71.2, R16.2
- net N$25: now also L10.2, U2.WCLK/GIO6; no longer L9.2, U1.WCLK/GIO6
- net N$26: now also C63.1, U4.BYPASS; no longer C33.1, U9.BYPASS
- net N$27: now also U2.AD1/GIO8; no longer U1.AD1/GIO8
- net N$28: now also R4.1, U2.GIO3; no longer R5.1, U1.GIO3
- net N$29: now also R4.2; no longer R5.2
- net N$3: now also L7.1, U2.!RESET; no longer L4.1, U1.!RESET
- net N$30: now also C90.2, R32.1, U11.SNS3K; no longer C58.2, R33.1, U8.SNS3K
- net N$31: now also R12.1; no longer R3.1
- net N$32: now also U6.!CHG; no longer U6.!CHRG
- net N$33: now also R11.1; no longer R18.1
- net N$34: now also C68.1, C69.1, U10P.VDDCORE; no longer C42.1, C45.1, U4P.VDDCORE
- net N$35: now also U10X.PX37, U9.CLK_IN; no longer U3.CLK_IN, U4X.PX37
- net N$39: now also R17.1, U10M.D-_FS; no longer R6.1, U4M.D-_FS
- net N$4: now also U2.AD0/GIO7; no longer U1.AD0/GIO7
- net N$40: now also C66.1, R21.1, U4.OUTB; no longer C39.1, R15.1, U9.OUTB
- net N$41: now also C91.2, R33.1, U11.SNS4K; no longer C59.2, R34.1, U8.SNS4K
- net N$42: now also C92.2, R34.1, U11.SNS5K; no longer C60.2, R35.1, U8.SNS5K
- net N$43: now also C87.2, R29.1, U11.SNS0K; no longer C30.2, R14.1, U8.SNS0K
- net N$45: now also C88.2, R30.1, U11.SNS1K; no longer C35.2, R28.1, U8.SNS1K
- net N$46: now also R15.1, U10M.D+_FS; no longer R17.1, U4M.D+_FS
- net N$47: now also C76.1, U10M.USB_VBIAS; no longer C72.1, U4M.USB_VBIAS
- net N$49: now also C67.1, R40.1; no longer C52.1, F1.1, L17.2, Q1.D, U6.VOUT, U6.VOUTS
- net N$5: now also L9.2, U2.BCLK/GIO5; no longer L6.2, U1.BCLK/GIO5
- net N$51: now also C52.1, R41.1; no longer Q1.G, U6.GATE
- net N$52: now also C83.1, U10C.PC02; no longer C75.1, U4C.PC02
- net N$53: now also R7.2, R9.1, U4.INA; no longer R12.2, R13.1, U9.INA
- net N$54: now also R14.1, R21.2, U4.INB; no longer R15.2, R16.1, U9.INB
- net N$55: now also R10.1, U4.SHUTDOWN; no longer R31.1, U9.SHUTDOWN
- net N$57: now also C84.1, U10C.PC03; no longer C73.1, U4C.PC03
- net N$58: now also Q4.D; no longer Q3.D
- net N$59: now also C87.1, U11.SNS0; no longer C30.1, U8.SNS0
- net N$60: now also C90.1, U11.SNS3; no longer C58.1, U8.SNS3
- net N$61: now also R32.2, VOL+.P$1; no longer R33.2, SW4.P$1
- net N$62: now also C91.1, U11.SNS4; no longer C59.1, U8.SNS4
- net N$63: now also R33.2, WIRELESS.P$1; no longer R34.2, SW5.P$1
- net N$64: now also C92.1, U11.SNS5; no longer C60.1, U8.SNS5
- net N$65: now also R34.2, VOL-.P$1; no longer R35.2, SW6.P$1
- net N$67: now also C54.1, L17.1, TO_AUX1.1, TO_AUX1.2; no longer C57.1, L19.1, TO_AUX2.1, TO_AUX2.2
- net N$7: now also R2.2, U1.BIAS; no longer R8.2, U2.BIAS
- net N$71: now also C93.2, R35.1, U11.SNS6K; no longer C61.2, R37.1, U8.SNS6K
- net N$72: now also PREV.P$1, R35.2; no longer R37.2, SW7.P$1
- net N$76: now also C93.1, U11.SNS6; no longer C61.1, U8.SNS6
- net N$77: now also R28.1, U11.!RESET; no longer R36.1, U8.!RESET
- net N$78: now also Q6.D; no longer Q4.D
- net N$79: now also Q3.D; no longer Q5.D
- net N$8: now also R1.1, U1.HGM; no longer R9.1, U2.HGM
- net N$80: now also Q5.D; no longer Q6.D
- net N$84: now also C62.1, L19.1, TO_AUX2.2, TO_AUX2.4; no longer C65.1, L18.1, TO_AUX1.2, TO_AUX1.4
- net N$85: now also R29.2, STOP.P$1; no longer R14.2, SW2.P$1
- net N$86: now also C88.1, U11.SNS1; no longer C35.1, U8.SNS1
- net N$87: now also NEXT.P$1, R30.2; no longer R28.2, SW3.P$1
- net N$88: now also C46.1, C47.1, U3.VQ; no longer C77.1, C78.1, U11.VQ
- net N$89: now also C44.1, C45.1, U3.FILT+; no longer C79.1, C80.1, U11.FILT+
- net N$9: now also C22.2; no longer C26.2
- net N$90: now also C89.2, R31.1, U11.SNS2K; no longer C43.2, R29.1, U8.SNS2K
- net N$91: now also C36.2, U3.AINA; no longer C81.2, U11.AINA
- net N$92: now also C38.2, U3.AINB; no longer C82.2, U11.AINB
- net N$93: now also C89.1, U11.SNS2; no longer C43.1, U8.SNS2
- net N$94: now also C82.1, U9.FILTP; no longer C101.1, U3.FILTP
- net N$95: now also BUTTON.P$1, R31.2; no longer R29.2, SW11.P$1
- net OUT_L: now also R41.2, U3.OUTB; no longer C70.1, U11.OUTB
- net OUT_R: now also R40.2, U3.OUTA; no longer C71.1, U11.OUTA
- net PA_EN: now also R6.2, U1.PAEN; no longer R10.2, U2.PAEN
- net PHONE_L: now also C53.2; no longer C36.2
- net PHONE_R: now also C66.2; no longer C39.2
- net PHONE_SENSE: now also R16.1, U10A.PA18; no longer R24.1, U4A.PA18
- net RED_BOT: now also TO_AUX1.4, U10A.PA12; no longer TO_AUX2.4, U4A.PA12
- net RED_TOP: now also TO_AUX1.7, U10X.PX17; no longer TO_AUX2.7, U4X.PX17
- net RTS: now also SERIAL.1, U10X.PX03; no longer U4X.PX03
- net RXD: now also SERIAL.3, U10X.PX00; no longer U4X.PX00
- net SCLK0: now also U10A.PA08, U2.SCLK, U3.SCL/SCLK, U9.SCL/SCLK; no longer TO_AUX1.1, U1.SCLK, U11.SCL/SCLK, U4A.PA08
- net SCLK1: now also TO_AUX2.1, U10B.PB07; no longer MICROSD.SCLK, U3.SCL/SCLK, U4B.PB07
- net TCK: now also U10M.TCK; no longer U4M.TCK
- net TDI: now also U10M.TDI; no longer U4M.TDI
- net TDO: now also U10M.TDO; no longer U4M.TDO
- net TMS: now also U10M.TMS; no longer U4M.TMS
- net TXD: now also SERIAL.2, U10X.PX01; no longer U4X.PX01
- net UC_MCLK: now also U10C.PC04, U8.!Q, U8.D; no longer U12.!Q, U12.D, U4C.PC04
- net USBOTGID: now also U10B.PB05; no longer U4B.PB05
- net VBUS: now also C59.1, U10P.USB_VBUS, U6.IN; no longer C51.1, R18.2, U4P.USB_VBUS, U6.D0, U6.VBUS
- net WCLK: now also L10.1, U10X.PX26, U10X.PX27, U10X.PX36, U3.WCLK; no longer L9.1, U11.WCLK, U4X.PX26, U4X.PX27, U4X.PX36
Other:
- note removed: "Configured to start on With Ilim = 1A"
- moved on the sheet: C1, C10, C11, C12, C13, C14, C15, C16, C17, C18, C19, C2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

Commit message: Minor revisions
Connections:
- net BCLK: no longer U10X.PX35
Changed lines of the file:
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@@
-</segment>
-<segment>
-<pinref part="U10" gate="X" pin="PX35"/>
-<wire x1="900.43" y1="-280.67" x2="905.51" y2="-280.67" width="0.1524" layer="91"/>
-<label x="905.51" y="-280.67" size="1.778" layer="95" xref="yes"/>
 </segment>
 <segment>
