File: draft11_proto.brd (EAGLE design)
At the start: 105 x 100 mm, 222 parts, among them Q2 2N7002, Q3 2N7002, Q4 2N7002, Q5 2N7002, Q6 2N7002, Q7 2N7002, U1 CC2591, U10 AT32UC3A3-LQFP-144, U11 AT42QT1110-QFN-32, U12 NAND-S34ML01G10TSOP-48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

Commit message: PCB work
Routed SDRAM, removed NAND
Parts:
- removed C27, C37: 100n, 00-EvaLibrary:C0603
- removed Q3, Q5, Q7: 2N7002, SparkFun-DiscreteSemi:SOT23-3
- removed U12: NAND-S34ML01G10TSOP-48, 00-EvaLibrary:TSOP-48
- added R10, R23, R42: 220, 00-EvaLibrary:R0603
- moved SERIAL 107.3 mm to (-81.5, -25.0), turned to 90 degrees
- moved C31 59.5 mm to (-86.8, -48.2), flipped to the top
- moved C45 59.5 mm to (-86.8, -46.2), flipped to the top
- moved C47 59.5 mm to (-86.8, -44.2), flipped to the top
- moved L15 59.5 mm to (-86.8, -50.2), flipped to the top
- moved C30 54.8 mm to (-83.5, -49.2), flipped to the top
- moved C44 54.8 mm to (-83.5, -47.2), flipped to the top
- moved C46 54.8 mm to (-83.5, -45.2), flipped to the top
- moved U3 46.6 mm to (-77.0, -47.2), flipped to the top
- moved C102 41.8 mm to (-61.8, -44.5), turned to 0 degrees
- moved C28 41.4 mm to (-71.2, -46.2), flipped to the top
- moved C29 41.4 mm to (-71.2, -48.2), flipped to the top
- moved C83 39.6 mm to (-61.8, -42.5), turned to 0 degrees
- moved C101 34.6 mm to (-61.8, -37.5), turned to 0 degrees
- moved C103 31.1 mm to (-61.8, -33.5), turned to 0 degrees
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Connections:
- removed net !CS_NAND: U10.42, U12.9
- removed net !RE: U10.39, U12.8
- removed net !WE_NAND: U10.56, U12.18
- removed net !WP: U10.57, U12.19
- removed net ALE: U10.79, U12.17
- removed net AUX_BLUE_BOT: Q7.1, TO_MAIN2.7
- removed net AUX_BLUE_TOP: Q6.1, TO_MAIN2.4
- removed net AUX_GREEN_BOT: Q5.1, TO_MAIN2.5
- removed net AUX_GREEN_TOP: Q4.1, TO_MAIN2.6
- removed net AUX_RED_BOT: Q3.1, TO_MAIN2.3
- removed net AUX_RED_TOP: Q2.1, TO_MAIN2.8
- removed net BLUE_BOT: TO_AUX1.8, U10.139
- removed net CLE: U10.78, U12.16
- removed net GREEN_BOT: TO_AUX1.6, U10.134
- removed net GREEN_TOP: TO_AUX1.5, U10.32
- removed net N$79: LED_LL.1, LED_LL.1-2, LED_LR.1, LED_LR.1-2, Q3.3
- removed net N$80: LED_LL.4, LED_LL.4-2, LED_LR.4, LED_LR.4-2, Q5.3
- removed net N$83: LED_LL.3, LED_LL.3-2, LED_LR.3, LED_LR.3-2, Q7.3
- removed net RDY/!BSY: U10.41, U12.7
- removed net RED_BOT: TO_AUX1.4, U10.132
- removed net RED_TOP: TO_AUX1.7, U10.15
- new net AUX_BLUE: R42.1, TO_MAIN2.4
- new net AUX_GREEN: R23.1, TO_MAIN2.6
- new net AUX_RED: R10.1, TO_MAIN2.8
- new net BLUE: TO_AUX1.7, U10.139
- new net GREEN: TO_AUX1.5, U10.134
- new net N$2: Q2.1, R10.2
- new net N$23: Q4.1, R23.2
- new net N$35: Q6.1, R42.2
- new net RED: TO_AUX1.3, U10.132
- net AUX_VSS1: now also TO_MAIN2.3, TO_MAIN2.5, TO_MAIN2.7; no longer Q3.2, Q5.2, Q7.2
- net BLUE_TOP: no longer TO_AUX1.3
- net D0: no longer U12.29
- net D1: no longer U12.30
- net D10: no longer U12.28
- net D11: no longer U12.33
- net D12: no longer U12.40
- net D13: no longer U12.45
- net D14: no longer U12.46
- net D15: no longer U12.47
- net D2: no longer U12.31
- net D3: no longer U12.32
- net D3.3V: no longer C27.1, C37.1, U12.12, U12.34, U12.37, U12.39
- net D4: no longer U12.41
- net D5: no longer U12.42
- net D6: no longer U12.43
- net D7: no longer U12.44
- net D8: no longer U12.26
- net D9: no longer U12.27
- net DGND: now also TO_AUX1.4, TO_AUX1.6, TO_AUX1.8; no longer C27.2, C37.2, U12.13, U12.25, U12.36, U12.48
- net N$56: now also LED_LL.1, LED_LL.1-2, LED_LR.1, LED_LR.1-2
- net N$58: now also LED_LL.4, LED_LL.4-2, LED_LR.4, LED_LR.4-2
- net N$78: now also LED_LL.3, LED_LL.3-2, LED_LR.3, LED_LR.3-2
Routing:
- net AUX_VDD2: track 242.9 -> 3.18 mm, vias 5 -> 0
- net N$58: track 215.9 -> 1.51 mm, vias 2 -> 0
- net N$56: track 216.5 -> 3.03 mm
- net N$78: track 211.5 -> 1.51 mm, vias 4 -> 0
- net ALE: track 61.6 -> 0.00 mm, vias 1 -> 0
- net N$79: track 60.2 -> 0.00 mm, vias 3 -> 0
- net CLE: track 58.4 -> 0.00 mm, vias 1 -> 0
- net N$83: track 50.3 -> 0.00 mm, vias 2 -> 0
- net N$80: track 45.3 -> 0.00 mm, vias 2 -> 0
- net !WP: track 44.9 -> 0.00 mm, vias 1 -> 0
- net !WE_NAND: track 43.0 -> 0.00 mm, vias 1 -> 0
- net D7: track 55.0 -> 19.8 mm
- net AUX_VSS1: track 36.9 -> 4.75 mm
- net D6: track 49.0 -> 19.9 mm
- net !CS_NAND: track 29.0 -> 0.00 mm, vias 1 -> 0
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