File: draft11_proto.sch (EAGLE design)
At the start: 213 parts, among them Q2 2N7002, Q3 2N7002, Q4 2N7002, Q5 2N7002, Q6 2N7002, Q7 2N7002, U1 CC2591, U10 AT32UC3A3-LQFP-144, U11 AT42QT1110-QFN-32, U12 NAND-S34ML01G10TSOP-48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

Commit message: PCB work
Routed SDRAM, removed NAND
Parts:
- removed C27, C37: 100n, 00-EvaLibrary:C-EUC0603
- removed Q3, Q5, Q7: 2N7002, SparkFun-DiscreteSemi:MOSFET-NCHANNELSMD
- removed U12: NAND-S34ML01G10TSOP-48, 00-EvaLibrary:NAND-S34ML01G10TSOP-48
- added R10, R23, R42: 220, 00-EvaLibrary:R-US_R0603
Connections:
- removed net !CS_NAND: U10X.PX53, U12.!CE
- removed net !RE: U10X.PX47, U12.!RE
- removed net !WE_NAND: U10X.PX59, U12.!WE
- removed net !WP: U10X.PX58, U12.!WP
- removed net ALE: U10X.PX55, U12.ALE
- removed net AUX_BLUE_BOT: Q7.G, TO_MAIN2.7
- removed net AUX_BLUE_TOP: Q6.G, TO_MAIN2.4
- removed net AUX_GREEN_BOT: Q5.G, TO_MAIN2.5
- removed net AUX_GREEN_TOP: Q4.G, TO_MAIN2.6
- removed net AUX_RED_BOT: Q3.G, TO_MAIN2.3
- removed net AUX_RED_TOP: Q2.G, TO_MAIN2.8
- removed net BLUE_BOT: TO_AUX1.8, U10A.PA09
- removed net CLE: U10X.PX56, U12.CLE
- removed net GREEN_BOT: TO_AUX1.6, U10B.PB06
- removed net GREEN_TOP: TO_AUX1.5, U10X.PX16
- removed net N$79: LED_LL.KR, LED_LR.KR, Q3.D
- removed net N$80: LED_LL.KG, LED_LR.KG, Q5.D
- removed net N$83: LED_LL.KB, LED_LR.KB, Q7.D
- removed net RDY/!BSY: U10X.PX48, U12.RDY/!BSY
- removed net RED_BOT: TO_AUX1.4, U10A.PA12
- removed net RED_TOP: TO_AUX1.7, U10A.PA02
- new net AUX_BLUE: R42.1, TO_MAIN2.4
- new net AUX_GREEN: R23.1, TO_MAIN2.6
- new net AUX_RED: R10.1, TO_MAIN2.8
- new net BLUE: TO_AUX1.7, U10A.PA09
- new net GREEN: TO_AUX1.5, U10B.PB06
- new net N$2: Q2.G, R10.2
- new net N$23: Q4.G, R23.2
- new net N$35: Q6.G, R42.2
- new net RED: TO_AUX1.3, U10A.PA12
- net AUX_VSS1: now also TO_MAIN2.3, TO_MAIN2.5, TO_MAIN2.7; no longer Q3.S, Q5.S, Q7.S
- net BLUE_TOP: no longer TO_AUX1.3
- net D0: no longer U12.IO0
- net D1: no longer U12.IO1
- net D10: no longer U12.IO10
- net D11: no longer U12.IO11
- net D12: no longer U12.IO12
- net D13: no longer U12.IO13
- net D14: no longer U12.IO14
- net D15: no longer U12.IO15
- net D2: no longer U12.IO2
- net D3: no longer U12.IO3
- net D3.3V: no longer C27.1, C37.1, U12.VDD
- net D4: no longer U12.IO4
- net D5: no longer U12.IO5
- net D6: no longer U12.IO6
- net D7: no longer U12.IO7
- net D8: no longer U12.IO8
- net D9: no longer U12.IO9
- net DGND: now also TO_AUX1.4, TO_AUX1.6, TO_AUX1.8; no longer C27.2, C37.2, U12.VSS
- net N$56: now also LED_LL.KR, LED_LR.KR
- net N$58: now also LED_LL.KG, LED_LR.KG
- net N$78: now also LED_LL.KB, LED_LR.KB
